File: covox.brd (EAGLE design)
At the start: 80 x 50 mm, 24 parts, among them CN1 POWERJACK, IC1 74HCT373N

Commit message: updates
Parts:
- added IC2: 74HC164N, 74xx-eu:DIL14
- C1: value 10uF -> 0.01uF
- C2: value (none) -> 0.1uF
- R10, R11, R12, R13, R14, R15, R16, R9: value 7.5k -> 7k5
- moved C1 23.2 mm to (62.2, 36.8), turned to 270 degrees
- moved R8 18.2 mm to (61.0, 14.0)
- moved JP3 18.2 mm to (66.0, 41.9)
- moved R16 17.3 mm to (67.3, 20.3), turned to 90 degrees
- moved C2 16.5 mm to (67.3, 30.5)
- moved R7 15.5 mm to (58.4, 16.5)
- moved R15 13.1 mm to (64.8, 20.3), turned to 270 degrees
- moved R6 12.8 mm to (55.9, 19.1)
- moved IC1 12.0 mm to (25.4, 12.7)
- moved R14 10.2 mm to (62.2, 22.9), turned to 270 degrees
- moved R5 10.2 mm to (53.3, 21.6)
- moved R4 7.73 mm to (50.8, 24.1)
- moved R13 7.41 mm to (59.7, 25.4), turned to 270 degrees
- moved R17 6.35 mm to (43.2, 34.3)
- moved R3 5.68 mm to (48.3, 26.7)
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Connections:
- removed net N$16: C1.2, C2.+, R16.2
- new net AOUT: C1.1, C2.+, R16.2
- net GND: now also C1.2, IC2.7; no longer C1.1
- net N$18: now also IC2.3
- net N$19: now also IC2.4
- net N$20: now also IC2.5
- net N$21: now also IC2.6
- net N$22: now also IC2.10
- net N$23: now also IC2.11
- net N$24: now also IC2.12
- net N$25: now also IC2.13
- net VCC: now also IC2.14
Routing:
- added copper zone on layer 16, net GND

Commit message: Updates...
Parts:
- C1: value 0.01uF -> 100nF; device rcl:C025-025X050 -> rcl:E2-4
- C2: value 0.1uF -> 10nF; device rcl:E2-4 -> rcl:C025-025X050
- R10, R12, R14, R16: value 7k5 -> 15k
- R17, R3, R5, R7: value 15k -> 7k5
- moved R17 27.9 mm to (67.3, 20.3), turned to 90 degrees
- moved R7 14.5 mm to (54.6, 30.5), turned to 270 degrees
- moved R8 14.4 mm to (50.8, 24.1)
- moved R10 11.5 mm to (53.3, 21.6), turned to 0 degrees
- moved R5 11.5 mm to (52.1, 33.0), turned to 270 degrees
- moved R6 10.8 mm to (48.3, 26.7)
- moved R9 10.8 mm to (57.1, 27.9)
- moved R16 8.98 mm to (61.0, 14.0), turned to 0 degrees
- moved R3 8.98 mm to (49.5, 35.6), turned to 270 degrees
- moved R12 8.98 mm to (55.9, 19.1), turned to 0 degrees
- moved C1 8.13 mm to (67.3, 30.5), turned to 90 degrees
- moved C2 8.13 mm to (62.2, 36.8), turned to 270 degrees
- moved R14 7.41 mm to (58.4, 16.5), turned to 0 degrees
- moved R11 7.18 mm to (59.7, 25.4)
- moved R4 7.18 mm to (45.7, 29.2)
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Connections:
- net AOUT: now also C1.+, C2.1, R17.2; no longer C1.1, C2.+, R16.2
- net GND: now also C2.2, R1.2; no longer C1.2, R17.2
- net N$1: now also R1.1, R2.2, R3.1; no longer R1.2, R17.1, R9.1
- net N$10: now also R6.1; no longer R3.1
- net N$11: now also R8.1; no longer R4.1
- net N$12: now also R10.1; no longer R5.1
- net N$13: now also R12.1; no longer R6.1
- net N$14: now also R14.1; no longer R7.1
- net N$15: now also R16.1; no longer R8.1
- net N$17: now also R16.2, R17.1; no longer R16.1, R8.2
- net N$2: now also R3.2, R4.2, R5.1; no longer R10.1, R2.2, R9.2
- net N$28: now also C1.-; no longer C2.-
- net N$3: now also R5.2, R6.2, R7.1; no longer R10.2, R11.1, R3.2
- net N$4: now also R7.2, R8.2, R9.1; no longer R11.2, R12.1, R4.2
- net N$5: now also R10.2, R11.1, R9.2; no longer R12.2, R13.1, R5.2
- net N$6: now also R11.2, R12.2, R13.1; no longer R13.2, R14.1, R6.2
- net N$7: now also R13.2; no longer R7.2
- net N$8: now also R2.1; no longer R1.1
- net N$9: now also R4.1; no longer R2.1

Commit message: Updates...
Parts:
- moved C2 3.81 mm to (66.0, 36.8), turned to 90 degrees
- moved JP3 1.27 mm to (67.3, 41.9)
- turned C1 to 0 degrees
Changed lines of the file:
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@@
 </autorouter>
 <elements>
-<element name="C2" library="rcl" package="C025-025X050" value="10nF" x="62.23" y="36.83" rot="R270"/>
-<element name="C1" library="rcl" package="E2-4" value="100nF" x="67.31" y="30.48" rot="R90"/>
+<element name="C2" library="rcl" package="C025-025X050" value="10nF" x="66.04" y="36.83" rot="R90"/>
+<element name="C1" library="rcl" package="E2-4" value="100nF" x="67.31" y="30.48"/>
 <element name="CN1" library="KaiBader" package="POWERJACK" value="POWERJACK" x="-2.54" y="44.45" rot="R270"/>
 <element name="IC1" library="74xx-eu" package="DIL20" value="74HCT373N" x="25.4" y="12.7" rot="R180"/>
 <element name="JP1" library="pinhead" package="1X08" value="" x="3.81" y="22.86" rot="R270"/>
 <element name="JP2" library="pinhead" package="1X02" value="" x="3.81" y="7.62" rot="R270"/>
-<element name="JP3" library="pinhead" package="1X02" value="" x="66.04" y="41.91" rot="R180"/>
+<element name="JP3" library="pinhead" package="1X02" value="" x="67.31" y="41.91" rot="R180"/>
 <element name="R2" library="rcl" package="0204/7" value="15k" x="43.18" y="31.75"/>
 <element name="R5" library="rcl" package="0204/7" value="7k5" x="52.07" y="33.02" rot="R270"/>
@@
 <contactref element="R1" pad="2"/>
 <contactref element="C2" pad="2"/>
-<wire x1="62.23" y1="35.56" x2="64.77" y2="41.91" width="0" layer="19" extent="1-1"/>
-<wire x1="39.37" y1="34.29" x2="62.23" y2="35.56" width="0" layer="19" extent="1-1"/>
+<wire x1="66.04" y1="38.1" x2="66.04" y2="41.91" width="0" layer="19" extent="1-1"/>
+<wire x1="39.37" y1="34.29" x2="66.04" y2="38.1" width="0" layer="19" extent="1-1"/>
 <wire x1="17.78" y1="41.91" x2="39.37" y2="34.29" width="0" layer="19" extent="1-1"/>
 <wire x1="8.16" y1="39.75" x2="17.78" y2="41.91" width="0" layer="19" extent="1-1"/>
@@
 <contactref element="C2" pad="1"/>
 <contactref element="C1" pad="+"/>
-<wire x1="67.31" y1="29.464" x2="62.23" y2="38.1" width="0" layer="19" extent="1-1"/>
-<wire x1="67.31" y1="24.13" x2="67.31" y2="29.464" width="0" layer="19" extent="1-1"/>
+<wire x1="66.294" y1="30.48" x2="66.04" y2="35.56" width="0" layer="19" extent="1-1"/>
+<wire x1="67.31" y1="24.13" x2="66.294" y2="30.48" width="0" layer="19" extent="1-1"/>
 </signal>
 <signal name="N$18">
@@
 <contactref element="C1" pad="-"/>
 <contactref element="JP3" pad="1"/>
-<wire x1="67.31" y1="31.496" x2="67.31" y2="41.91" width="0" layer="19" extent="1-1"/>
+<wire x1="68.326" y1="30.48" x2="68.58" y2="41.91" width="0" layer="19" extent="1-1"/>
 </signal>
 </signals>

Commit message: Updates...
Parts:
- added R18: 47k (optional), rcl:0204/7
Connections:
- net GND: now also R18.1
- net N$28: now also R18.2
Changed lines of the file:
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@@
 <element name="R3" library="rcl" package="0204/7" value="7k5" x="49.53" y="35.56" rot="R270"/>
 <element name="IC2" library="74xx-eu" package="DIL14" value="74HC164N" x="25.4" y="38.1" rot="R180"/>
+<element name="R18" library="rcl" package="0204/7" value="47k (optional)" x="2.54" y="-5.08"/>
 </elements>
 <signals>
@@
 <contactref element="R1" pad="2"/>
 <contactref element="C2" pad="2"/>
+<contactref element="R18" pad="1"/>
 <wire x1="66.04" y1="38.1" x2="66.04" y2="41.91" width="0" layer="19" extent="1-1"/>
 <wire x1="39.37" y1="34.29" x2="66.04" y2="38.1" width="0" layer="19" extent="1-1"/>
@@
 <wire x1="5.16" y1="44.45" x2="8.16" y2="39.75" width="0" layer="19" extent="1-1"/>
 <wire x1="13.97" y1="16.51" x2="8.16" y2="39.75" width="0" layer="19" extent="1-1"/>
+<wire x1="-1.27" y1="-5.08" x2="13.97" y2="16.51" width="0" layer="19" extent="1-1"/>
 </signal>
 <signal name="VCC" class="1">
@@
 <contactref element="C1" pad="-"/>
 <contactref element="JP3" pad="1"/>
+<contactref element="R18" pad="2"/>
 <wire x1="68.326" y1="30.48" x2="68.58" y2="41.91" width="0" layer="19" extent="1-1"/>
+<wire x1="6.35" y1="-5.08" x2="68.326" y2="30.48" width="0" layer="19" extent="1-1"/>
 </signal>
 </signals>

Commit message: Updates...
Parts:
- IC1: value 74HCT373N -> 74HC164N; device 74xx-eu:DIL20 -> 74xx-eu:DIL14
- IC2: value 74HC164N -> 74HCT373N; device 74xx-eu:DIL14 -> 74xx-eu:DIL20
- R10, R12, R14, R16: value 15k -> 7k5
- R3, R5, R7, R9: value 7k5 -> 15k
- moved R18 78.6 mm to (67.3, 39.4)
- moved IC1 25.4 mm to (25.4, 38.1)
- moved IC2 25.4 mm to (25.4, 12.7)
- moved R10 14.5 mm to (49.5, 35.6), turned to 270 degrees
- moved R9 14.5 mm to (61.0, 14.0), turned to 0 degrees
- moved R12 11.5 mm to (54.6, 30.5), turned to 270 degrees
- moved R7 11.5 mm to (55.9, 19.1), turned to 0 degrees
- moved R11 10.8 mm to (52.1, 33.0)
- moved R8 10.8 mm to (58.4, 16.5)
- moved R5 8.98 mm to (50.8, 24.1), turned to 0 degrees
- moved R14 8.98 mm to (59.7, 25.4), turned to 270 degrees
- moved R3 7.41 mm to (45.7, 29.2), turned to 0 degrees
- moved R16 7.41 mm to (64.8, 20.3), turned to 270 degrees
- moved R6 7.18 mm to (53.3, 21.6)
- moved R13 7.18 mm to (57.1, 27.9)
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Connections:
- net GND: now also IC1.7, IC2.10, R1.1; no longer IC1.10, IC2.7, R1.2
- net N$1: now also R1.2, R10.1; no longer R1.1, R3.1
- net N$10: now also IC2.6, R4.1; no longer IC1.6, R6.1
- net N$11: now also IC2.9, R5.1; no longer IC1.9, R8.1
- net N$12: now also IC2.12, R6.1; no longer IC1.12, R10.1
- net N$13: now also IC2.15, R7.1; no longer IC1.15, R12.1
- net N$14: now also IC2.16, R8.1; no longer IC1.16, R14.1
- net N$15: now also IC2.19, R9.1; no longer IC1.19, R16.1
- net N$17: now also R9.2; no longer R15.2
- net N$2: now also R10.2, R11.1; no longer R4.2, R5.1
- net N$20: now also IC1.5, IC2.7; no longer IC1.7, IC2.5
- net N$21: now also IC1.6, IC2.8; no longer IC1.8, IC2.6
- net N$22: now also IC1.10, IC2.13; no longer IC1.13, IC2.10
- net N$23: now also IC1.11, IC2.14; no longer IC1.14, IC2.11
- net N$24: now also IC1.12, IC2.17; no longer IC1.17, IC2.12
- net N$25: now also IC1.13, IC2.18; no longer IC1.18, IC2.13
- net N$26: now also IC2.1; no longer IC1.1
- net N$27: now also IC2.11; no longer IC1.11
- net N$3: now also R11.2, R12.1, R4.2; no longer R5.2, R6.2, R7.1
- net N$4: now also R12.2, R13.1, R5.2; no longer R7.2, R8.2, R9.1
- net N$5: now also R13.2, R14.1, R6.2; no longer R10.2, R11.1, R9.2
- net N$6: now also R14.2, R15.1, R7.2; no longer R11.2, R12.2, R13.1
- net N$7: now also R15.2, R16.1, R8.2; no longer R13.2, R14.2, R15.1
- net N$8: now also IC2.2; no longer IC1.2
- net N$9: now also IC2.5, R3.1; no longer IC1.5, R4.1
- net VCC: now also IC1.14, IC2.20; no longer IC1.20, IC2.14

Commit message: Updates...
Parts:
- added JP4: SER-IN, pinhead:1X04
- JP1: value (none) -> PAR-IN
- JP2: value (none) -> LATCH
- moved CN1 85.9 mm to (68.6, -3.81), turned to 0 degrees
- moved JP2 30.7 mm to (34.3, 3.81), turned to 180 degrees
- moved R10 26.2 mm to (25.4, 45.7)
- moved R17 26.2 mm to (43.2, 30.5)
- moved R6 26.2 mm to (29.2, 31.8)
- moved R7 26.2 mm to (31.8, 29.2)
- moved R8 26.2 mm to (34.3, 26.7)
- moved R9 26.2 mm to (36.8, 24.1)
- moved R1 26.2 mm to (19.1, 44.5)
- moved R11 26.2 mm to (27.9, 43.2)
- moved R12 26.2 mm to (30.5, 40.6)
- moved R14 26.2 mm to (35.6, 35.6)
- moved R15 26.2 mm to (38.1, 33.0)
- moved R2 26.2 mm to (19.1, 41.9)
- moved R3 26.2 mm to (21.6, 39.4)
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Connections:
- new net N$16: IC1.1, JP4.1
- new net N$29: IC1.2, JP4.2
- new net N$30: IC1.9, JP4.4
- new net N$31: IC1.8, JP4.3

Commit message: Updates...
Parts:
- moved CN1 35.2 mm to (53.3, 27.9), turned to 90 degrees
- moved JP3 28.2 mm to (47.0, 45.7)
- moved R18 26.7 mm to (43.2, 43.2)
- moved C2 25.4 mm to (39.4, 43.2), turned to 0 degrees
- moved C1 19.7 mm to (39.4, 47.0), turned to 0 degrees
- moved R13 14.0 mm to (19.1, 38.1)
- moved R14 14.0 mm to (21.6, 35.6)
- moved R15 14.0 mm to (24.1, 33.0)
- moved R5 14.0 mm to (12.7, 34.3)
- moved R1 14.0 mm to (5.08, 44.5)
- moved R11 14.0 mm to (14.0, 43.2)
- moved R2 14.0 mm to (5.08, 41.9)
- moved R6 14.0 mm to (15.2, 31.8)
- moved R10 14.0 mm to (11.4, 45.7)
- moved R12 14.0 mm to (16.5, 40.6)
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Routing:
- added copper zone on layer 1, net GND
Other:
- board size 80 x 50 mm -> 50 x 50 mm
