File: covox.brd (EAGLE design)
At the start: 50 x 50 mm, 27 parts, among them CN1 POWERJACK, IC1 74HC164N, IC2 74HCT373N

Commit message: updates
Parts:
- added JP5: (no value), SparkFun-Connectors:STEREOJACK2.5MM_SPECIA_POGOPINS
- moved R16 15.3 mm to (20.3, 44.5), turned to 90 degrees
- moved R17 15.3 mm to (22.9, 44.5)
- moved R15 13.1 mm to (17.8, 44.5), turned to 90 degrees
- moved R14 10.9 mm to (15.2, 44.5), turned to 90 degrees
- moved R1 10.5 mm to (2.54, 34.3), turned to 90 degrees
- moved R9 10.2 mm to (22.9, 34.3), turned to 90 degrees
- moved R13 8.98 mm to (12.7, 44.5), turned to 90 degrees
- moved R2 7.62 mm to (5.08, 34.3), turned to 90 degrees
- moved R8 7.62 mm to (20.3, 34.3), turned to 90 degrees
- moved R12 7.41 mm to (10.2, 44.5), turned to 90 degrees
- moved R11 6.48 mm to (7.62, 44.5), turned to 90 degrees
- moved R10 6.48 mm to (5.08, 44.5), turned to 90 degrees
- moved R3 5.08 mm to (7.62, 34.3), turned to 90 degrees
- moved R7 5.08 mm to (17.8, 34.3), turned to 90 degrees
- moved C2 2.54 mm to (39.4, 40.6), turned to 270 degrees
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Connections:
- removed net N$28: C1.-, JP3.1, R18.2
- new net N$32: C1.-, JP3.1, JP5.SHIELD, JP5.TIP, R18.2
- net GND: now also JP5.RING1

Commit message: updates
Parts:
- added U$1: (no value), KaiBader-Various:COVOX_LOGO
- moved R18 1.27 mm to (43.2, 43.2)
- moved CN1 1.27 mm to (53.3, 27.9)
- moved C1 0.90 mm to (38.7, 46.4)
- moved R15 0.64 mm to (17.1, 44.5)
- moved R16 0.64 mm to (19.7, 44.5)
- moved R5 0.64 mm to (13.3, 34.3)
- moved R9 0.64 mm to (23.5, 34.3)
- moved R3 0.64 mm to (8.26, 34.3)
- moved R1 0.63 mm to (3.17, 34.3)
- moved R10 0.63 mm to (4.45, 44.5)
- moved R11 0.63 mm to (6.99, 44.5)
- moved R12 0.63 mm to (9.53, 44.5)
- moved R13 0.63 mm to (12.1, 44.5)
- moved R14 0.63 mm to (14.6, 44.5)
- moved R2 0.63 mm to (5.71, 34.3)
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Other:
- board text added: "CC-BY-SA 4.0 2015 KAI C. BADER"

Commit message: updates
Parts:
- removed U$1: (no value), KaiBader-Various:COVOX_LOGO
- added U$2: (no value), KaiBader-Various:COVOX_LOGO_600
Changed lines of the file:
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@@
 <element name="JP4" library="pinhead" package="1X04" value="SER-IN" x="43.18" y="3.81"/>
 <element name="JP5" library="SparkFun-Connectors" package="STEREOJACK2.5MM_SPECIA_POGOPINS" value="" x="30.48" y="44.45" rot="R270"/>
-<element name="U$1" library="KaiBader-Various" package="COVOX_LOGO" value="" x="2.54" y="22.225"/>
+<element name="U$2" library="KaiBader-Various" package="COVOX_LOGO_600" value="" x="3.175" y="22.225"/>
 </elements>
 <signals>
