File: covox.brd (EAGLE design)
At the start: 50 x 50 mm, 29 parts, among them CN1 POWERJACK, IC1 74HCT164, IC2 74HCT373

Commit message: update
Parts:
- JP3: value (none) -> SER-IN; device pinhead:1X02 -> pinhead:1X05
- JP4: value SER-IN -> (none); device pinhead:1X04 -> SparkFun-Connectors:STEREOJACK2.5MM_SPECIA_POGOPINS
- JP5: device SparkFun-Connectors:STEREOJACK2.5MM_SPECIA_POGOPINS -> pinhead:1X02
- moved JP4 42.6 mm to (30.5, 44.5), turned to 270 degrees
- moved JP3 39.8 mm to (41.9, 3.81), turned to 0 degrees
- moved JP5 17.2 mm to (47.6, 43.2)
- moved JP2 1.27 mm to (29.2, 3.81)
Connections:
- net GND: now also JP4.RING1, JP5.2; no longer JP3.2, JP5.RING1
- net N$16: now also JP3.2; no longer JP4.1
- net N$29: now also JP3.3; no longer JP4.2
- net N$30: now also JP3.5; no longer JP4.4
- net N$31: now also JP3.4; no longer JP4.3
- net N$32: now also JP4.SHIELD, JP4.TIP, JP5.1; no longer JP3.1, JP5.SHIELD, JP5.TIP
Routing:
- net N$21: track 117.5 -> 0.00 mm
- net N$23: track 82.9 -> 0.00 mm, vias 1 -> 0
- net VCC: track 66.3 -> 0.00 mm, vias 1 -> 0
- net N$22: track 65.0 -> 0.00 mm, vias 3 -> 0
- net N$19: track 51.9 -> 0.00 mm, vias 1 -> 0
- net N$24: track 46.6 -> 0.00 mm, vias 2 -> 0
- net N$25: track 44.3 -> 0.00 mm
- net N$18: track 37.7 -> 0.00 mm
- net N$20: track 33.8 -> 0.00 mm, vias 1 -> 0
- net N$15: track 32.4 -> 0.00 mm
- net N$32: track 30.7 -> 0.00 mm
- net AOUT: track 29.4 -> 0.00 mm
- net N$26: track 29.0 -> 0.00 mm
- net N$11: track 24.9 -> 0.00 mm
- net N$12: track 22.4 -> 0.00 mm
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Other:
- board text added: "VCC"

Commit message: updates
Parts:
- removed JP4: (no value), SparkFun-Connectors:STEREOJACK2.5MM_SPECIA_POGOPINS
- added JP6: (no value), KaiBader:AUDIO-JACK-3.5MM
- moved JP5 18.8 mm to (29.2, 47.0), turned to 0 degrees
- moved R18 14.0 mm to (29.2, 42.5), turned to 180 degrees
- moved C1 12.6 mm to (29.2, 38.1), turned to 0 degrees
- moved C2 12.2 mm to (29.2, 33.0), turned to 0 degrees
- moved U$2 1.91 mm to (2.54, 23.5)
Connections:
- net GND: now also JP6.1; no longer JP4.RING1
- net N$32: now also JP6.2, JP6.3; no longer JP4.SHIELD, JP4.TIP
Other:
- board text added: "GND"
- board text added: "SPK"
Changed lines of the file:
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@@
 <wire x1="50" y1="50" x2="0" y2="50" width="0" layer="20"/>
 <wire x1="0" y1="50" x2="0" y2="0" width="0" layer="20"/>
-<text x="32.385" y="34.29" size="1.27" layer="21" font="vector" ratio="12" align="center">CC-BY-SA 4.0
-2015
-KAI C. BADER</text>
+<text x="2.54" y="21.59" size="1.27" layer="21" font="vector" ratio="12">CC-BY-SA 4.0  2015  KAI C. BADER</text>
 <text x="1.905" y="44.45" size="1.27" layer="25" font="vector" ratio="12" rot="R270" align="bottom-center">7k5 x8</text>
 <text x="0.635" y="34.29" size="1.27" layer="25" font="vector" ratio="12" rot="R270" align="bottom-center">15k x9</text>
@@
 <text x="6.985" y="5.715" size="1.27" layer="27" font="vector" ratio="12" rot="R90">D6</text>
 <text x="4.445" y="5.715" size="1.27" layer="27" font="vector" ratio="12" rot="R90">D7</text>
-<text x="43.815" y="43.18" size="1.27" layer="27" font="vector" ratio="12" rot="R90" align="bottom-center">(opt)</text>
+<text x="29.21" y="43.18" size="1.27" layer="27" font="vector" ratio="12" rot="R180" align="bottom-center">(opt)</text>
 <text x="37.465" y="5.715" size="1.27" layer="27" font="vector" ratio="12" rot="R90">VCC</text>
 <wire x1="36.83" y1="8.89" x2="36.83" y2="9.525" width="0.1524" layer="27"/>
 <wire x1="36.83" y1="9.525" x2="39.37" y2="9.525" width="0.1524" layer="27"/>
 <wire x1="39.37" y1="9.525" x2="39.37" y2="6.985" width="0.1524" layer="27"/>
+<text x="26.035" y="45.72" size="1.27" layer="27" font="vector" ratio="12" rot="R90">SPK</text>
+<text x="33.655" y="45.72" size="1.27" layer="27" font="vector" ratio="12" rot="R90">GND</text>
 </plain>
 <attributes>
@@
 </autorouter>
 <elements>
-<element name="C2" library="rcl" package="C025-025X050" value="10nF" x="38.735" y="40.64" smashed="yes" rot="R270">
-<attribute name="VALUE" x="41.275" y="40.64" size="1.27" layer="27" font="vector" ratio="12" rot="R90" align="bottom-center"/>
-</element>
-<element name="C1" library="rcl" package="E2-4" value="100nF" x="38.735" y="46.355" smashed="yes" rot="R90">
-<attribute name="VALUE" x="34.925" y="46.355" size="1.27" layer="27" font="vector" ratio="12" rot="R270" align="bottom-center"/>
+<element name="C2" library="rcl" package="C025-025X050" value="10nF" x="29.21" y="33.02" smashed="yes">
+<attribute name="VALUE" x="32.385" y="33.02" size="1.27" layer="27" font="vector" ratio="12" rot="R270" align="bottom-center"/>
+</element>
+<element name="C1" library="rcl" package="E2-4" value="100nF" x="29.21" y="38.1" smashed="yes">
+<attribute name="VALUE" x="25.4" y="38.1" size="1.27" layer="27" font="vector" ratio="12" rot="R270" align="bottom-center"/>
 </element>
 <element name="CN1" library="KaiBader" package="POWERJACK" value="POWERJACK" x="53.34" y="27.94" smashed="yes" rot="R90"/>
@@
 <attribute name="VALUE" x="29.21" y="1.27" size="1.27" layer="27" font="vector" ratio="12" align="center"/>
 </element>
-<element name="JP5" library="pinhead" package="1X02" value="" x="47.625" y="43.18" smashed="yes" rot="R270">
-<attribute name="VALUE" x="44.45" y="45.72" size="1.27" layer="27" rot="R270"/>
+<element name="JP5" library="pinhead" package="1X02" value="" x="29.21" y="46.99" smashed="yes">
+<attribute name="VALUE" x="26.67" y="43.815" size="1.27" layer="27"/>
 </element>
 <element name="R2" library="rcl" package="0204/7" value="15k" x="5.715" y="34.29" smashed="yes" rot="R90"/>
@@
 <attribute name="VALUE" x="39.37" y="15.24" size="1.27" layer="27" font="vector" ratio="12" align="center"/>
 </element>
-<element name="R18" library="rcl" package="0204/7" value="47k (optional)" x="43.18" y="43.18" smashed="yes" rot="R90"/>
-<element name="JP4" library="SparkFun-Connectors" package="STEREOJACK2.5MM_SPECIA_POGOPINS" value="" x="30.48" y="44.45" smashed="yes" rot="R270"/>
-<element name="U$2" library="KaiBader-Various" package="COVOX_LOGO_600" value="" x="4.445" y="23.495" smashed="yes"/>
+<element name="R18" library="rcl" package="0204/7" value="47k (optional)" x="29.21" y="42.545" smashed="yes" rot="R180"/>
+<element name="U$2" library="KaiBader-Various" package="COVOX_LOGO_600" value="" x="2.54" y="23.495" smashed="yes"/>
 <element name="JP3" library="pinhead" package="1X05" value="SER-IN" x="41.91" y="3.81" smashed="yes">
 <attribute name="VALUE" x="41.91" y="1.27" size="1.27" layer="27" ratio="12" align="center"/>
 </element>
+<element name="JP6" library="KaiBader" package="AUDIO-JACK-3.5MM" value="" x="49.53" y="48.26" rot="R180"/>
 </elements>
 <signals>
@@
 <vertex x="0" y="50"/>
 </polygon>
-<contactref element="JP4" pad="RING1"/>
-<wire x1="43.18" y1="39.37" x2="47.625" y2="41.91" width="0" layer="19" extent="1-1"/>
-<wire x1="38.735" y1="39.37" x2="43.18" y2="39.37" width="0" layer="19" extent="1-1"/>
-<wire x1="42.64" y1="32.64" x2="43.18" y2="39.37" width="0" layer="19" extent="1-1"/>
-<wire x1="45.64" y1="27.94" x2="42.64" y2="32.64" width="0" layer="19" extent="1-1"/>
-<wire x1="28.63" y1="41.95" x2="38.735" y2="39.37" width="0" layer="19" extent="1-1"/>
-<wire x1="46.99" y1="11.43" x2="45.64" y2="27.94" width="0" layer="19" extent="1-1"/>
-<wire x1="26.67" y1="11.43" x2="46.99" y2="11.43" width="0" layer="19" extent="1-1"/>
-<wire x1="3.175" y1="30.48" x2="28.63" y2="41.95" width="0" layer="19" extent="1-1"/>
+<contactref element="JP6" pad="1"/>
 </signal>
 <signal name="VCC" class="1">
@@
 <contactref element="C2" pad="1"/>
 <contactref element="C1" pad="+"/>
-<wire x1="38.735" y1="41.91" x2="38.735" y2="45.339" width="0" layer="19" extent="1-1"/>
-<wire x1="22.225" y1="48.26" x2="38.735" y2="45.339" width="0" layer="19" extent="1-1"/>
+<wire x1="28.194" y1="38.1" x2="22.225" y2="48.26" width="0" layer="19" extent="1-1"/>
+<wire x1="27.94" y1="33.02" x2="28.194" y2="38.1" width="0" layer="19" extent="1-1"/>
 </signal>
 <signal name="N$18">
@@
 </signal>
 <signal name="N$32">
-<contactref element="JP4" pad="TIP"/>
-<contactref element="JP4" pad="SHIELD"/>
 <contactref element="JP5" pad="1"/>
 <contactref element="C1" pad="-"/>
 <contactref element="R18" pad="2"/>
-<wire x1="43.18" y1="46.99" x2="47.625" y2="44.45" width="0" layer="19" extent="1-1"/>
-<wire x1="38.735" y1="47.371" x2="43.18" y2="46.99" width="0" layer="19" extent="1-1"/>
-<wire x1="30.48" y1="46.85" x2="38.735" y2="47.371" width="0" layer="19" extent="1-1"/>
-<wire x1="30.48" y1="39.95" x2="30.48" y2="46.85" width="0" layer="19" extent="1-1"/>
+<contactref element="JP6" pad="2"/>
+<contactref element="JP6" pad="3"/>
+<wire x1="39.43" y1="37.46" x2="44.23" y2="46.96" width="0" layer="19" extent="1-1"/>
+<wire x1="30.226" y1="38.1" x2="39.43" y2="37.46" width="0" layer="19" extent="1-1"/>
+<wire x1="25.4" y1="42.545" x2="30.226" y2="38.1" width="0" layer="19" extent="1-1"/>
+<wire x1="27.94" y1="46.99" x2="25.4" y2="42.545" width="0" layer="19" extent="1-1"/>
 </signal>
 </signals>
 </board>
 </drawing>
-<compatibility>
-<note version="6.3" minversion="6.2.2" severity="warning">
-Since Version 6.2.2 text objects can contain more than one line,
-which will not be processed correctly with this version.
-</note>
-</compatibility>
 </eagle>

Commit message: updates
Parts:
- turned C2 to 180 degrees
- turned JP5 to 180 degrees
- turned R18 to 0 degrees
Changed lines of the file:
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@@
 <wire x1="36.83" y1="9.525" x2="39.37" y2="9.525" width="0.1524" layer="27"/>
 <wire x1="39.37" y1="9.525" x2="39.37" y2="6.985" width="0.1524" layer="27"/>
-<text x="26.035" y="45.72" size="1.27" layer="27" font="vector" ratio="12" rot="R90">SPK</text>
-<text x="33.655" y="45.72" size="1.27" layer="27" font="vector" ratio="12" rot="R90">GND</text>
+<text x="33.655" y="45.72" size="1.27" layer="27" font="vector" ratio="12" rot="R90">SPK</text>
+<text x="26.035" y="45.72" size="1.27" layer="27" font="vector" ratio="12" rot="R90">GND</text>
 </plain>
 <attributes>
@@
 </autorouter>
 <elements>
-<element name="C2" library="rcl" package="C025-025X050" value="10nF" x="29.21" y="33.02" smashed="yes">
-<attribute name="VALUE" x="32.385" y="33.02" size="1.27" layer="27" font="vector" ratio="12" rot="R270" align="bottom-center"/>
+<element name="C2" library="rcl" package="C025-025X050" value="10nF" x="29.21" y="33.02" smashed="yes" rot="R180">
+<attribute name="VALUE" x="26.67" y="33.02" size="1.27" layer="27" font="vector" ratio="12" rot="R90" align="bottom-center"/>
 </element>
 <element name="C1" library="rcl" package="E2-4" value="100nF" x="29.21" y="38.1" smashed="yes">
-<attribute name="VALUE" x="25.4" y="38.1" size="1.27" layer="27" font="vector" ratio="12" rot="R270" align="bottom-center"/>
+<attribute name="VALUE" x="31.75" y="38.1" size="1.27" layer="27" font="vector" ratio="12" rot="R270" align="bottom-center"/>
 </element>
 <element name="CN1" library="KaiBader" package="POWERJACK" value="POWERJACK" x="53.34" y="27.94" smashed="yes" rot="R90"/>
@@
 <attribute name="VALUE" x="29.21" y="1.27" size="1.27" layer="27" font="vector" ratio="12" align="center"/>
 </element>
-<element name="JP5" library="pinhead" package="1X02" value="" x="29.21" y="46.99" smashed="yes">
-<attribute name="VALUE" x="26.67" y="43.815" size="1.27" layer="27"/>
+<element name="JP5" library="pinhead" package="1X02" value="" x="29.21" y="46.99" smashed="yes" rot="R180">
+<attribute name="VALUE" x="31.75" y="50.165" size="1.27" layer="27" rot="R180"/>
 </element>
 <element name="R2" library="rcl" package="0204/7" value="15k" x="5.715" y="34.29" smashed="yes" rot="R90"/>
@@
 <attribute name="VALUE" x="39.37" y="15.24" size="1.27" layer="27" font="vector" ratio="12" align="center"/>
 </element>
-<element name="R18" library="rcl" package="0204/7" value="47k (optional)" x="29.21" y="42.545" smashed="yes" rot="R180"/>
+<element name="R18" library="rcl" package="0204/7" value="47k (optional)" x="29.21" y="42.545" smashed="yes"/>
 <element name="U$2" library="KaiBader-Various" package="COVOX_LOGO_600" value="" x="2.54" y="23.495" smashed="yes"/>
 <element name="JP3" library="pinhead" package="1X05" value="SER-IN" x="41.91" y="3.81" smashed="yes">
@@
 <contactref element="C1" pad="+"/>
 <wire x1="28.194" y1="38.1" x2="22.225" y2="48.26" width="0" layer="19" extent="1-1"/>
-<wire x1="27.94" y1="33.02" x2="28.194" y2="38.1" width="0" layer="19" extent="1-1"/>
+<wire x1="30.48" y1="33.02" x2="28.194" y2="38.1" width="0" layer="19" extent="1-1"/>
 </signal>
 <signal name="N$18">
@@
 <contactref element="JP6" pad="3"/>
 <wire x1="39.43" y1="37.46" x2="44.23" y2="46.96" width="0" layer="19" extent="1-1"/>
-<wire x1="30.226" y1="38.1" x2="39.43" y2="37.46" width="0" layer="19" extent="1-1"/>
-<wire x1="25.4" y1="42.545" x2="30.226" y2="38.1" width="0" layer="19" extent="1-1"/>
-<wire x1="27.94" y1="46.99" x2="25.4" y2="42.545" width="0" layer="19" extent="1-1"/>
+<wire x1="33.02" y1="42.545" x2="39.43" y2="37.46" width="0" layer="19" extent="1-1"/>
+<wire x1="30.48" y1="46.99" x2="33.02" y2="42.545" width="0" layer="19" extent="1-1"/>
+<wire x1="30.226" y1="38.1" x2="33.02" y2="42.545" width="0" layer="19" extent="1-1"/>
 </signal>
 </signals>

Commit message: updates
Connections:
- net VCC: now also JP3.1
Routing:
- net N$24: track 0.00 -> 78.7 mm, vias 0 -> 1
- net VCC: track 0.00 -> 60.2 mm
- net N$21: track 0.00 -> 55.8 mm
- net N$25: track 0.00 -> 54.7 mm, vias 0 -> 2
- net N$18: track 0.00 -> 48.3 mm
- net N$22: track 0.00 -> 47.0 mm, vias 0 -> 2
- net N$19: track 0.00 -> 46.2 mm
- net N$23: track 0.00 -> 45.7 mm, vias 0 -> 2
- net N$20: track 0.00 -> 43.0 mm, vias 0 -> 3
- net N$11: track 0.00 -> 39.4 mm, vias 0 -> 2
- net N$32: track 0.00 -> 30.1 mm
- net N$10: track 0.00 -> 28.2 mm
- net N$26: track 0.00 -> 27.7 mm, vias 0 -> 1
- net N$12: track 0.00 -> 26.4 mm
- net N$15: track 0.00 -> 24.6 mm, vias 0 -> 1
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
Commit message: updates
Routing:
- net N$31: track 17.9 -> 24.6 mm
Changed lines of the file:
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@@
 <param name="PrefDir.14" value="0"/>
 <param name="PrefDir.15" value="0"/>
-<param name="PrefDir.16" value="*"/>
+<param name="PrefDir.16" value="|"/>
 <param name="cfVia" value="50"/>
 <param name="cfNonPref" value="5"/>
@@
 </polygon>
 <contactref element="JP6" pad="1"/>
+<via x="1.27" y="48.895" extent="1-16" drill="0.6096" diameter="0.9144"/>
+<via x="48.895" y="48.895" extent="1-16" drill="0.6096" diameter="0.9144"/>
+<via x="48.895" y="1.27" extent="1-16" drill="0.6096" diameter="0.9144"/>
+<via x="1.27" y="1.27" extent="1-16" drill="0.6096" diameter="0.9144"/>
+<via x="25.4" y="3.175" extent="1-16" drill="0.6096" diameter="0.9144"/>
+<via x="34.29" y="1.27" extent="1-16" drill="0.6096" diameter="0.9144"/>
+<via x="34.925" y="5.715" extent="1-16" drill="0.6096" diameter="0.9144"/>
+<via x="19.05" y="8.89" extent="1-16" drill="0.6096" diameter="0.9144"/>
+<via x="25.4" y="29.845" extent="1-16" drill="0.6096" diameter="0.9144"/>
+<via x="13.335" y="27.305" extent="1-16" drill="0.6096" diameter="0.9144"/>
+<via x="9.525" y="26.035" extent="1-16" drill="0.6096" diameter="0.9144"/>
+<via x="5.715" y="27.305" extent="1-16" drill="0.6096" diameter="0.9144"/>
+<via x="29.845" y="26.035" extent="1-16" drill="0.6096" diameter="0.9144"/>
+<via x="24.765" y="40.005" extent="1-16" drill="0.6096" diameter="0.9144"/>
+<via x="1.905" y="40.005" extent="1-16" drill="0.6096" diameter="0.9144"/>
+<via x="29.845" y="20.32" extent="1-16" drill="0.6096" diameter="0.9144"/>
 </signal>
 <signal name="VCC" class="1">
@@
 <contactref element="IC1" pad="8"/>
 <contactref element="JP3" pad="4"/>
-<wire x1="46.9392" y1="17.0688" x2="46.9392" y2="19.05" width="0.3048" layer="16"/>
-<wire x1="48.768" y1="15.24" x2="46.9392" y2="17.0688" width="0.3048" layer="16"/>
-<wire x1="48.768" y1="9.4488" x2="48.768" y2="15.24" width="0.3048" layer="16"/>
-<wire x1="44.5008" y1="5.1816" x2="48.768" y2="9.4488" width="0.3048" layer="16"/>
-<wire x1="44.5008" y1="3.81" x2="44.5008" y2="5.1816" width="0.3048" layer="16"/>
-<wire x1="46.9392" y1="19.05" x2="46.99" y2="19.05" width="0.3048" layer="16"/>
-<wire x1="44.5008" y1="3.81" x2="44.45" y2="3.81" width="0.3048" layer="16"/>
+<wire x1="47.3964" y1="18.7452" x2="47.0916" y2="19.05" width="0.3048" layer="1"/>
+<wire x1="47.3964" y1="18.5928" x2="47.3964" y2="18.7452" width="0.3048" layer="1"/>
+<wire x1="48.768" y1="17.2212" x2="47.3964" y2="18.5928" width="0.3048" layer="1"/>
+<wire x1="48.768" y1="14.9352" x2="48.768" y2="17.2212" width="0.3048" layer="1"/>
+<wire x1="49.3776" y1="14.3256" x2="48.768" y2="14.9352" width="0.3048" layer="1"/>
+<wire x1="49.3776" y1="3.048" x2="49.3776" y2="14.3256" width="0.3048" layer="1"/>
+<wire x1="47.3964" y1="1.0668" x2="49.3776" y2="3.048" width="0.3048" layer="1"/>
+<wire x1="46.482" y1="1.0668" x2="47.3964" y2="1.0668" width="0.3048" layer="1"/>
+<wire x1="46.3296" y1="1.2192" x2="46.482" y2="1.0668" width="0.3048" layer="1"/>
+<wire x1="45.8724" y1="1.2192" x2="46.3296" y2="1.2192" width="0.3048" layer="1"/>
+<wire x1="44.5008" y1="2.5908" x2="45.8724" y2="1.2192" width="0.3048" layer="1"/>
+<wire x1="44.5008" y1="3.81" x2="44.5008" y2="2.5908" width="0.3048" layer="1"/>
+<wire x1="47.0916" y1="19.05" x2="46.99" y2="19.05" width="0.3048" layer="1"/>
+<wire x1="44.5008" y1="3.81" x2="44.45" y2="3.81" width="0.3048" layer="1"/>
 </signal>
 <signal name="N$32">
@@
 <wire x1="44.196" y1="46.9392" x2="44.23" y2="46.96" width="0.3048" layer="1"/>
 </signal>
-<signal name="N$28">
-<via x="1.27" y="48.895" extent="1-16" drill="0.6" diameter="1.016"/>
-</signal>
-<signal name="N$33">
-<via x="48.895" y="48.895" extent="1-16" drill="0.6" diameter="1.016"/>
-</signal>
-<signal name="N$34">
-<via x="48.895" y="1.27" extent="1-16" drill="0.6" diameter="1.016"/>
-</signal>
 </signals>

Commit message: updates
Parts:
- added JP4: PWR, pinhead:1X02
- JP5: device pinhead:1X02 -> KaiBader:AUDIO-JACK-3.5MM
- JP6: value (none) -> AUDIO; device KaiBader:AUDIO-JACK-3.5MM -> pinhead:1X02
- moved JP5 20.4 mm to (49.5, 48.3)
- moved JP6 20.4 mm to (29.2, 47.0)
- moved U$2 1.27 mm to (1.27, 23.5)
Connections:
- net GND: now also JP4.2, JP5.1, JP6.2; no longer JP5.2, JP6.1
- net N$32: now also JP5.2, JP5.3, JP6.1; no longer JP5.1, JP6.2, JP6.3
- net VCC: now also JP4.1
Routing:
- net N$24: track 78.7 -> 0.00 mm, vias 1 -> 0
- net VCC: track 60.2 -> 0.00 mm
- net N$21: track 55.8 -> 0.00 mm
- net N$25: track 54.7 -> 0.00 mm, vias 2 -> 0
- net N$18: track 48.3 -> 0.00 mm
- net N$22: track 47.0 -> 0.00 mm, vias 2 -> 0
- net N$19: track 46.2 -> 0.00 mm
- net N$23: track 45.7 -> 0.00 mm, vias 2 -> 0
- net N$20: track 43.0 -> 0.00 mm, vias 3 -> 0
- net N$11: track 39.4 -> 0.00 mm, vias 2 -> 0
- net N$32: track 30.1 -> 0.00 mm
- net N$10: track 28.2 -> 0.00 mm
- net N$26: track 27.7 -> 0.00 mm, vias 1 -> 0
- net N$12: track 26.4 -> 0.00 mm
- net N$31: track 24.6 -> 0.00 mm
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Other:
- board text added: "CC-BY-SA 4.0 KAI C. BADER"
- board text removed: "CC-BY-SA 4.0 2015 KAI C. BADER"

Commit message: updates
Routing:
- net N$24: track 0.00 -> 79.4 mm, vias 0 -> 1
- net VCC: track 0.00 -> 63.9 mm
- net N$25: track 0.00 -> 56.6 mm, vias 0 -> 2
- net N$21: track 0.00 -> 55.8 mm
- net N$18: track 0.00 -> 48.3 mm
- net N$23: track 0.00 -> 46.2 mm, vias 0 -> 1
- net N$19: track 0.00 -> 46.2 mm
- net N$22: track 0.00 -> 45.2 mm, vias 0 -> 2
- net N$20: track 0.00 -> 43.0 mm, vias 0 -> 3
- net N$11: track 0.00 -> 39.8 mm, vias 0 -> 2
- net N$32: track 0.00 -> 30.1 mm
- net N$10: track 0.00 -> 28.2 mm
- net N$26: track 0.00 -> 27.7 mm, vias 0 -> 1
- net N$12: track 0.00 -> 26.7 mm
- net N$31: track 0.00 -> 24.9 mm
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
Commit message: updates
Parts:
- JP2: device pinhead:1X02 -> pinhead:1X03
Connections:
- net GND: now also JP2.1
- net N$26: now also JP2.2; no longer JP2.1
- net N$27: now also JP2.3; no longer JP2.2
Routing:
- net N$20: track 43.0 -> 35.9 mm, vias 3 -> 1
- net N$18: track 48.3 -> 50.3 mm, vias 0 -> 1
- net N$26: track 27.7 -> 29.6 mm
- net N$21: track 55.8 -> 54.0 mm
- net N$27: track 16.8 -> 17.4 mm
Other:
- board text added: "OE"
- board text removed: "OC"
