File: covox.sch (EAGLE design)
At the start: 24 parts, among them CN1 POWERJACK, IC1 74HCT373N

Commit message: updates
Parts:
- added IC2: 74HC164N, 74xx-eu:74HC164N
- C1: value 10uF -> 0.01uF
- C2: value (none) -> 0.1uF
- R10, R11, R12, R13, R14, R15, R16, R9: value 7.5k -> 7k5
Connections:
- removed net N$16: C1.2, C2.+, R16.2
- new net AOUT: C1.1, C2.+, R16.2
- net GND: now also C1.2; no longer C1.1
- net N$18: now also IC2A.QA
- net N$19: now also IC2A.QB
- net N$20: now also IC2A.QC
- net N$21: now also IC2A.QD
- net N$22: now also IC2A.QE
- net N$23: now also IC2A.QF
- net N$24: now also IC2A.QG
- net N$25: now also IC2A.QH
Other:
- moved on the sheet: C1, C2, IC1, JP3, R1, R10, R11, R12, R13, R14, R15, R16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

Commit message: Updates...
Parts:
- C1: value 0.01uF -> 100nF; device rcl:C-EU025-025X050 -> rcl:CPOL-EUE2-4
- C2: value 0.1uF -> 10nF; device rcl:CPOL-EUE2-4 -> rcl:C-EU025-025X050
- R10, R12, R14, R16: value 7k5 -> 15k
- R17, R3, R5, R7: value 15k -> 7k5
Connections:
- net AOUT: now also C1.+, C2.1, R17.2; no longer C1.1, C2.+, R16.2
- net GND: now also C2.2, R1.2; no longer C1.2, R17.2
- net N$1: now also R1.1, R2.2, R3.1; no longer R1.2, R17.1, R9.1
- net N$10: now also R6.1; no longer R3.1
- net N$11: now also R8.1; no longer R4.1
- net N$12: now also R10.1; no longer R5.1
- net N$13: now also R12.1; no longer R6.1
- net N$14: now also R14.1; no longer R7.1
- net N$15: now also R16.1; no longer R8.1
- net N$17: now also R16.2, R17.1; no longer R16.1, R8.2
- net N$2: now also R3.2, R4.2, R5.1; no longer R10.1, R2.2, R9.2
- net N$28: now also C1.-; no longer C2.-
- net N$3: now also R5.2, R6.2, R7.1; no longer R10.2, R11.1, R3.2
- net N$4: now also R7.2, R8.2, R9.1; no longer R11.2, R12.1, R4.2
- net N$5: now also R10.2, R11.1, R9.2; no longer R12.2, R13.1, R5.2
- net N$6: now also R11.2, R12.2, R13.1; no longer R13.2, R14.1, R6.2
- net N$7: now also R13.2; no longer R7.2
- net N$8: now also R2.1; no longer R1.1
- net N$9: now also R4.1; no longer R2.1
Other:
- moved on the sheet: R1, R10, R11, R12, R13, R14, R16, R17, R2, R3, R4, R5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

Commit message: Updates...
Parts:
- added R18: 47k (optional), rcl:R-EU_0204/7
Connections:
- net GND: now also R18.1
- net N$28: now also R18.2
Other:
- moved on the sheet: C1, C2, IC1, IC2, JP3, R1, R10, R11, R12, R13, R14, R15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

Commit message: Updates...
Parts:
- IC1: value 74HCT373N -> 74HC164N; device 74xx-eu:74HCT373N -> 74xx-eu:74HC164N
- IC2: value 74HC164N -> 74HCT373N; device 74xx-eu:74HC164N -> 74xx-eu:74HCT373N
- R10, R12, R14, R16: value 15k -> 7k5
- R3, R5, R7, R9: value 7k5 -> 15k
Connections:
- net GND: now also R1.1; no longer R1.2
- net N$1: now also R1.2, R10.1; no longer R1.1, R3.1
- net N$10: now also IC2A.3Q, R4.1; no longer IC1A.3Q, R6.1
- net N$11: now also IC2A.4Q, R5.1; no longer IC1A.4Q, R8.1
- net N$12: now also IC2A.5Q, R6.1; no longer IC1A.5Q, R10.1
- net N$13: now also IC2A.6Q, R7.1; no longer IC1A.6Q, R12.1
- net N$14: now also IC2A.7Q, R8.1; no longer IC1A.7Q, R14.1
- net N$15: now also IC2A.8Q, R9.1; no longer IC1A.8Q, R16.1
- net N$17: now also R9.2; no longer R15.2
- net N$18: now also IC1A.QA, IC2A.1D; no longer IC1A.1D, IC2A.QA
- net N$19: now also IC1A.QB, IC2A.2D; no longer IC1A.2D, IC2A.QB
- net N$2: now also R10.2, R11.1; no longer R4.2, R5.1
- net N$20: now also IC1A.QC, IC2A.3D; no longer IC1A.3D, IC2A.QC
- net N$21: now also IC1A.QD, IC2A.4D; no longer IC1A.4D, IC2A.QD
- net N$22: now also IC1A.QE, IC2A.5D; no longer IC1A.5D, IC2A.QE
- net N$23: now also IC1A.QF, IC2A.6D; no longer IC1A.6D, IC2A.QF
- net N$24: now also IC1A.QG, IC2A.7D; no longer IC1A.7D, IC2A.QG
- net N$25: now also IC1A.QH, IC2A.8D; no longer IC1A.8D, IC2A.QH
- net N$26: now also IC2A.OC; no longer IC1A.OC
- net N$27: now also IC2A.ENC; no longer IC1A.ENC
- net N$3: now also R11.2, R12.1, R4.2; no longer R5.2, R6.2, R7.1
- net N$4: now also R12.2, R13.1, R5.2; no longer R7.2, R8.2, R9.1
- net N$5: now also R13.2, R14.1, R6.2; no longer R10.2, R11.1, R9.2
- net N$6: now also R14.2, R15.1, R7.2; no longer R11.2, R12.2, R13.1
- net N$7: now also R15.2, R16.1, R8.2; no longer R13.2, R14.2, R15.1
- net N$8: now also IC2A.1Q; no longer IC1A.1Q
- net N$9: now also IC2A.2Q, R3.1; no longer IC1A.2Q, R4.1
Other:
- moved on the sheet: R1, R10, R11, R12, R13, R14, R15, R16, R3, R4, R5, R6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

Commit message: Updates...
Parts:
- added JP4: SER-IN, pinhead:PINHD-1X4
- JP1: value (none) -> PAR-IN
- JP2: value (none) -> LATCH
Connections:
- new net N$16: IC1A.A, JP4.1
- new net N$29: IC1A.B, JP4.2
- new net N$30: IC1A.CLR, JP4.4
- new net N$31: IC1A.CLK, JP4.3
Other:
- moved on the sheet: JP2
Changed lines of the file:
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@@
 <part name="C2" library="rcl" deviceset="C-EU" device="025-025X050" value="10nF"/>
 <part name="C1" library="rcl" deviceset="CPOL-EU" device="E2-4" value="100nF"/>
-<part name="JP1" library="pinhead" deviceset="PINHD-1X8" device=""/>
-<part name="JP2" library="pinhead" deviceset="PINHD-1X2" device=""/>
+<part name="JP1" library="pinhead" deviceset="PINHD-1X8" device="" value="PAR-IN"/>
+<part name="JP2" library="pinhead" deviceset="PINHD-1X2" device="" value="LATCH"/>
 <part name="JP3" library="pinhead" deviceset="PINHD-1X2" device=""/>
 <part name="CN1" library="KaiBader" deviceset="POWERJACK" device=""/>
@@
 <part name="IC1" library="74xx-eu" deviceset="74*164" device="N" technology="HC"/>
 <part name="R18" library="rcl" deviceset="R-EU_" device="0204/7" value="47k (optional)"/>
+<part name="JP4" library="pinhead" deviceset="PINHD-1X4" device="" value="SER-IN"/>
 </parts>
 <sheets>
@@
 <instance part="C1" gate="G$1" x="185.42" y="22.86" rot="R90"/>
 <instance part="JP1" gate="A" x="-2.54" y="66.04" rot="MR0"/>
-<instance part="JP2" gate="G$1" x="-2.54" y="45.72" rot="MR0"/>
+<instance part="JP2" gate="G$1" x="-2.54" y="43.18" rot="MR0"/>
 <instance part="JP3" gate="G$1" x="213.36" y="20.32"/>
 <instance part="CN1" gate="G$1" x="7.62" y="106.68"/>
@@
 <instance part="IC1" gate="A" x="30.48" y="22.86"/>
 <instance part="R18" gate="G$1" x="195.58" y="17.78" rot="R90"/>
+<instance part="JP4" gate="A" x="-2.54" y="25.4" rot="MR0"/>
 </instances>
 <busses>
@@
 <segment>
 <pinref part="JP2" gate="G$1" pin="1"/>
-<wire x1="0" y1="48.26" x2="12.7" y2="48.26" width="0.1524" layer="91"/>
-<wire x1="12.7" y1="48.26" x2="12.7" y2="53.34" width="0.1524" layer="91"/>
+<wire x1="0" y1="45.72" x2="12.7" y2="45.72" width="0.1524" layer="91"/>
+<wire x1="12.7" y1="45.72" x2="12.7" y2="53.34" width="0.1524" layer="91"/>
 <pinref part="IC2" gate="A" pin="OC"/>
 <wire x1="12.7" y1="53.34" x2="83.82" y2="53.34" width="0.1524" layer="91"/>
@@
 <segment>
 <pinref part="JP2" gate="G$1" pin="2"/>
-<wire x1="0" y1="45.72" x2="15.24" y2="45.72" width="0.1524" layer="91"/>
-<wire x1="15.24" y1="45.72" x2="15.24" y2="50.8" width="0.1524" layer="91"/>
+<wire x1="0" y1="43.18" x2="15.24" y2="43.18" width="0.1524" layer="91"/>
+<wire x1="15.24" y1="43.18" x2="15.24" y2="50.8" width="0.1524" layer="91"/>
 <pinref part="IC2" gate="A" pin="ENC"/>
 <wire x1="15.24" y1="50.8" x2="83.82" y2="50.8" width="0.1524" layer="91"/>
@@
 </segment>
 </net>
+<net name="N$16" class="0">
+<segment>
+<pinref part="JP4" gate="A" pin="1"/>
+<pinref part="IC1" gate="A" pin="A"/>
+<wire x1="0" y1="30.48" x2="17.78" y2="30.48" width="0.1524" layer="91"/>
+</segment>
+</net>
+<net name="N$29" class="0">
+<segment>
+<pinref part="JP4" gate="A" pin="2"/>
+<pinref part="IC1" gate="A" pin="B"/>
+<wire x1="0" y1="27.94" x2="17.78" y2="27.94" width="0.1524" layer="91"/>
+</segment>
+</net>
+<net name="N$30" class="0">
+<segment>
+<pinref part="JP4" gate="A" pin="4"/>
+<wire x1="0" y1="22.86" x2="12.7" y2="22.86" width="0.1524" layer="91"/>
+<wire x1="12.7" y1="22.86" x2="12.7" y2="12.7" width="0.1524" layer="91"/>
+<pinref part="IC1" gate="A" pin="CLR"/>
+<wire x1="12.7" y1="12.7" x2="17.78" y2="12.7" width="0.1524" layer="91"/>
+</segment>
+</net>
+<net name="N$31" class="0">
+<segment>
+<pinref part="IC1" gate="A" pin="CLK"/>
+<wire x1="17.78" y1="17.78" x2="15.24" y2="17.78" width="0.1524" layer="91"/>
+<wire x1="15.24" y1="17.78" x2="15.24" y2="25.4" width="0.1524" layer="91"/>
+<pinref part="JP4" gate="A" pin="3"/>
+<wire x1="15.24" y1="25.4" x2="0" y2="25.4" width="0.1524" layer="91"/>
+</segment>
+</net>

Commit message: updates
Parts:
- added JP5: (no value), SparkFun-Connectors:AUDIO-JACKSPECIAL_POGO_PINS
Connections:
- removed net N$28: C1.-, JP3.1, R18.2
- new net N$32: C1.-, JP3.1, JP5.LEFT, JP5.RIGHT, R18.2
- net GND: now also JP5.SLEEVE
Other:
- moved on the sheet: JP3
Changed lines of the file:
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@@
 <part name="R18" library="rcl" deviceset="R-EU_" device="0204/7" value="47k (optional)"/>
 <part name="JP4" library="pinhead" deviceset="PINHD-1X4" device="" value="SER-IN"/>
+<part name="JP5" library="SparkFun-Connectors" deviceset="AUDIO-JACK" device="SPECIAL_POGO_PINS"/>
 </parts>
 <sheets>
@@
 <instance part="JP1" gate="A" x="-2.54" y="66.04" rot="MR0"/>
 <instance part="JP2" gate="G$1" x="-2.54" y="43.18" rot="MR0"/>
-<instance part="JP3" gate="G$1" x="213.36" y="20.32"/>
+<instance part="JP3" gate="G$1" x="223.52" y="20.32"/>
 <instance part="CN1" gate="G$1" x="7.62" y="106.68"/>
 <instance part="P+1" gate="VCC" x="20.32" y="121.92"/>
@@
 <instance part="R18" gate="G$1" x="195.58" y="17.78" rot="R90"/>
 <instance part="JP4" gate="A" x="-2.54" y="25.4" rot="MR0"/>
+<instance part="JP5" gate="G$1" x="218.44" y="40.64" rot="MR0"/>
 </instances>
 <busses>
@@
 <pinref part="JP3" gate="G$1" pin="2"/>
 <pinref part="GND3" gate="1" pin="GND"/>
-<wire x1="210.82" y1="20.32" x2="203.2" y2="20.32" width="0.1524" layer="91"/>
+<wire x1="220.98" y1="20.32" x2="203.2" y2="20.32" width="0.1524" layer="91"/>
 <wire x1="203.2" y1="20.32" x2="203.2" y2="12.7" width="0.1524" layer="91"/>
 <pinref part="C2" gate="G$1" pin="2"/>
@@
 <wire x1="195.58" y1="12.7" x2="203.2" y2="12.7" width="0.1524" layer="91"/>
 <junction x="195.58" y="12.7"/>
+<wire x1="203.2" y1="20.32" x2="203.2" y2="43.18" width="0.1524" layer="91"/>
+<junction x="203.2" y="20.32"/>
+<pinref part="JP5" gate="G$1" pin="SLEEVE"/>
+<wire x1="203.2" y1="43.18" x2="213.36" y2="43.18" width="0.1524" layer="91"/>
 </segment>
 <segment>
@@
 </segment>
 </net>
-<net name="N$28" class="0">
-<segment>
-<pinref part="C1" gate="G$1" pin="-"/>
-<pinref part="JP3" gate="G$1" pin="1"/>
-<wire x1="190.5" y1="22.86" x2="195.58" y2="22.86" width="0.1524" layer="91"/>
-<pinref part="R18" gate="G$1" pin="2"/>
-<wire x1="195.58" y1="22.86" x2="210.82" y2="22.86" width="0.1524" layer="91"/>
-<junction x="195.58" y="22.86"/>
-</segment>
-</net>
 <net name="VCC" class="1">
 <segment>
@@
 </segment>
 </net>
+<net name="N$32" class="0">
+<segment>
+<pinref part="JP5" gate="G$1" pin="RIGHT"/>
+<pinref part="JP5" gate="G$1" pin="LEFT"/>
+<wire x1="213.36" y1="40.64" x2="213.36" y2="38.1" width="0.1524" layer="91"/>
+<pinref part="C1" gate="G$1" pin="-"/>
+<pinref part="JP3" gate="G$1" pin="1"/>
+<wire x1="190.5" y1="22.86" x2="195.58" y2="22.86" width="0.1524" layer="91"/>
+<pinref part="R18" gate="G$1" pin="2"/>
+<wire x1="195.58" y1="22.86" x2="205.74" y2="22.86" width="0.1524" layer="91"/>
+<junction x="195.58" y="22.86"/>
+<wire x1="205.74" y1="22.86" x2="220.98" y2="22.86" width="0.1524" layer="91"/>
+<wire x1="213.36" y1="38.1" x2="205.74" y2="38.1" width="0.1524" layer="91"/>
+<wire x1="205.74" y1="38.1" x2="205.74" y2="22.86" width="0.1524" layer="91"/>
+<junction x="213.36" y="38.1"/>
+<junction x="205.74" y="22.86"/>
+</segment>
+</net>

Commit message: updates
Other:
- moved on the sheet: CN1
Changed lines of the file:
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@@
 <instance part="JP2" gate="G$1" x="-2.54" y="43.18" rot="MR0"/>
 <instance part="JP3" gate="G$1" x="223.52" y="20.32"/>
-<instance part="CN1" gate="G$1" x="7.62" y="106.68"/>
-<instance part="P+1" gate="VCC" x="20.32" y="121.92"/>
-<instance part="GND1" gate="1" x="20.32" y="96.52"/>
+<instance part="CN1" gate="G$1" x="215.9" y="66.04" rot="MR0"/>
+<instance part="P+1" gate="VCC" x="203.2" y="81.28" rot="MR0"/>
+<instance part="GND1" gate="1" x="203.2" y="60.96" rot="MR0"/>
 <instance part="GND2" gate="1" x="119.38" y="81.28"/>
-<instance part="GND3" gate="1" x="203.2" y="2.54"/>
+<instance part="GND3" gate="1" x="203.2" y="5.08"/>
 <instance part="IC1" gate="A" x="30.48" y="22.86"/>
 <instance part="R18" gate="G$1" x="195.58" y="17.78" rot="R90"/>
@@
 <wire x1="203.2" y1="20.32" x2="203.2" y2="12.7" width="0.1524" layer="91"/>
 <pinref part="C2" gate="G$1" pin="2"/>
-<wire x1="203.2" y1="12.7" x2="203.2" y2="5.08" width="0.1524" layer="91"/>
+<wire x1="203.2" y1="12.7" x2="203.2" y2="7.62" width="0.1524" layer="91"/>
 <wire x1="190.5" y1="12.7" x2="195.58" y2="12.7" width="0.1524" layer="91"/>
 <junction x="203.2" y="12.7"/>
@@
 <pinref part="CN1" gate="G$1" pin="GNDBREAK"/>
 <pinref part="CN1" gate="G$1" pin="GND"/>
-<wire x1="10.16" y1="111.76" x2="10.16" y2="109.22" width="0.1524" layer="91"/>
+<wire x1="213.36" y1="71.12" x2="213.36" y2="68.58" width="0.1524" layer="91"/>
 <pinref part="GND1" gate="1" pin="GND"/>
-<wire x1="10.16" y1="109.22" x2="20.32" y2="109.22" width="0.1524" layer="91"/>
-<wire x1="20.32" y1="109.22" x2="20.32" y2="99.06" width="0.1524" layer="91"/>
-<junction x="10.16" y="109.22"/>
+<wire x1="213.36" y1="68.58" x2="203.2" y2="68.58" width="0.1524" layer="91"/>
+<wire x1="203.2" y1="68.58" x2="203.2" y2="63.5" width="0.1524" layer="91"/>
+<junction x="213.36" y="68.58"/>
 </segment>
 <segment>
@@
 <pinref part="CN1" gate="G$1" pin="PWR"/>
 <pinref part="P+1" gate="VCC" pin="VCC"/>
-<wire x1="10.16" y1="114.3" x2="20.32" y2="114.3" width="0.1524" layer="91"/>
-<wire x1="20.32" y1="114.3" x2="20.32" y2="119.38" width="0.1524" layer="91"/>
-</segment>
-</net>
+<wire x1="213.36" y1="73.66" x2="203.2" y2="73.66" width="0.1524" layer="91"/>
+<wire x1="203.2" y1="73.66" x2="203.2" y2="78.74" width="0.1524" layer="91"/>
+</segment>
+</net>

Commit message: updates
Parts:
- IC1: value 74HC164N -> 74HCT164
- IC2: value 74HCT373N -> 74HCT373
Changed lines of the file:
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@@
 </classes>
 <parts>
-<part name="IC2" library="74xx-eu" deviceset="74*373" device="N" technology="HCT"/>
+<part name="IC2" library="74xx-eu" deviceset="74*373" device="N" technology="HCT" value="74HCT373"/>
 <part name="R2" library="rcl" deviceset="R-EU_" device="0204/7" value="15k"/>
 <part name="R3" library="rcl" deviceset="R-EU_" device="0204/7" value="15k"/>
@@
 <part name="GND2" library="supply1" deviceset="GND" device=""/>
 <part name="GND3" library="supply1" deviceset="GND" device=""/>
-<part name="IC1" library="74xx-eu" deviceset="74*164" device="N" technology="HC"/>
+<part name="IC1" library="74xx-eu" deviceset="74*164" device="N" technology="HC" value="74HCT164"/>
 <part name="R18" library="rcl" deviceset="R-EU_" device="0204/7" value="47k (optional)"/>
 <part name="JP4" library="pinhead" deviceset="PINHD-1X4" device="" value="SER-IN"/>
