File: covox.sch (EAGLE design)
At the start: 28 parts, among them CN1 POWERJACK, IC1 74HCT164, IC2 74HCT373

Commit message: update
Parts:
- JP3: value (none) -> SER-IN; device pinhead:PINHD-1X2 -> pinhead:PINHD-1X5
- JP4: value SER-IN -> (none); device pinhead:PINHD-1X4 -> SparkFun-Connectors:AUDIO-JACKSPECIAL_POGO_PINS
- JP5: device SparkFun-Connectors:AUDIO-JACKSPECIAL_POGO_PINS -> pinhead:PINHD-1X2
Connections:
- net GND: now also JP4.SLEEVE, JP5.2; no longer JP3.2, JP5.SLEEVE
- net N$16: now also JP3.2; no longer JP4.1
- net N$29: now also JP3.3; no longer JP4.2
- net N$30: now also JP3.5; no longer JP4.4
- net N$31: now also JP3.4; no longer JP4.3
- net N$32: now also JP4.LEFT, JP4.RIGHT, JP5.1; no longer JP3.1, JP5.LEFT, JP5.RIGHT
Other:
- moved on the sheet: IC1
Changed lines of the file:
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@@
 <part name="JP1" library="pinhead" deviceset="PINHD-1X8" device="" value="PAR-IN"/>
 <part name="JP2" library="pinhead" deviceset="PINHD-1X2" device="" value="LATCH"/>
-<part name="JP3" library="pinhead" deviceset="PINHD-1X2" device=""/>
+<part name="JP5" library="pinhead" deviceset="PINHD-1X2" device=""/>
 <part name="CN1" library="KaiBader" deviceset="POWERJACK" device=""/>
 <part name="P+1" library="supply1" deviceset="VCC" device=""/>
+<part name="GND2" library="supply1" deviceset="GND" device=""/>
 <part name="GND1" library="supply1" deviceset="GND" device=""/>
-<part name="GND2" library="supply1" deviceset="GND" device=""/>
 <part name="GND3" library="supply1" deviceset="GND" device=""/>
 <part name="IC1" library="74xx-eu" deviceset="74*164" device="N" technology="HC" value="74HCT164"/>
 <part name="R18" library="rcl" deviceset="R-EU_" device="0204/7" value="47k (optional)"/>
-<part name="JP4" library="pinhead" deviceset="PINHD-1X4" device="" value="SER-IN"/>
-<part name="JP5" library="SparkFun-Connectors" deviceset="AUDIO-JACK" device="SPECIAL_POGO_PINS"/>
+<part name="JP4" library="SparkFun-Connectors" deviceset="AUDIO-JACK" device="SPECIAL_POGO_PINS"/>
+<part name="JP3" library="pinhead" deviceset="PINHD-1X5" device="" value="SER-IN"/>
 </parts>
 <sheets>
@@
 <instance part="JP1" gate="A" x="-2.54" y="66.04" rot="MR0"/>
 <instance part="JP2" gate="G$1" x="-2.54" y="43.18" rot="MR0"/>
-<instance part="JP3" gate="G$1" x="223.52" y="20.32"/>
+<instance part="JP5" gate="G$1" x="223.52" y="20.32"/>
 <instance part="CN1" gate="G$1" x="215.9" y="66.04" rot="MR0"/>
 <instance part="P+1" gate="VCC" x="203.2" y="81.28" rot="MR0"/>
-<instance part="GND1" gate="1" x="203.2" y="60.96" rot="MR0"/>
-<instance part="GND2" gate="1" x="119.38" y="81.28"/>
+<instance part="GND2" gate="1" x="203.2" y="60.96" rot="MR0"/>
+<instance part="GND1" gate="1" x="119.38" y="81.28"/>
 <instance part="GND3" gate="1" x="203.2" y="5.08"/>
-<instance part="IC1" gate="A" x="30.48" y="22.86"/>
+<instance part="IC1" gate="A" x="30.48" y="20.32"/>
 <instance part="R18" gate="G$1" x="195.58" y="17.78" rot="R90"/>
-<instance part="JP4" gate="A" x="-2.54" y="25.4" rot="MR0"/>
-<instance part="JP5" gate="G$1" x="218.44" y="40.64" rot="MR0"/>
+<instance part="JP4" gate="G$1" x="218.44" y="40.64" rot="MR0"/>
+<instance part="JP3" gate="A" x="-2.54" y="25.4" rot="MR0"/>
 </instances>
 <busses>
@@
 <pinref part="IC1" gate="A" pin="QA"/>
 <wire x1="48.26" y1="76.2" x2="83.82" y2="76.2" width="0.1524" layer="91"/>
-<wire x1="43.18" y1="30.48" x2="48.26" y2="30.48" width="0.1524" layer="91"/>
-<wire x1="48.26" y1="30.48" x2="48.26" y2="76.2" width="0.1524" layer="91"/>
+<wire x1="43.18" y1="27.94" x2="48.26" y2="27.94" width="0.1524" layer="91"/>
+<wire x1="48.26" y1="27.94" x2="48.26" y2="76.2" width="0.1524" layer="91"/>
 <junction x="48.26" y="76.2"/>
 </segment>
@@
 <pinref part="IC1" gate="A" pin="QB"/>
 <wire x1="50.8" y1="73.66" x2="83.82" y2="73.66" width="0.1524" layer="91"/>
-<wire x1="43.18" y1="27.94" x2="50.8" y2="27.94" width="0.1524" layer="91"/>
-<wire x1="50.8" y1="27.94" x2="50.8" y2="73.66" width="0.1524" layer="91"/>
+<wire x1="43.18" y1="25.4" x2="50.8" y2="25.4" width="0.1524" layer="91"/>
+<wire x1="50.8" y1="25.4" x2="50.8" y2="73.66" width="0.1524" layer="91"/>
 <junction x="50.8" y="73.66"/>
 </segment>
@@
 <pinref part="IC1" gate="A" pin="QC"/>
 <wire x1="53.34" y1="71.12" x2="83.82" y2="71.12" width="0.1524" layer="91"/>
-<wire x1="43.18" y1="25.4" x2="53.34" y2="25.4" width="0.1524" layer="91"/>
-<wire x1="53.34" y1="25.4" x2="53.34" y2="71.12" width="0.1524" layer="91"/>
+<wire x1="43.18" y1="22.86" x2="53.34" y2="22.86" width="0.1524" layer="91"/>
+<wire x1="53.34" y1="22.86" x2="53.34" y2="71.12" width="0.1524" layer="91"/>
 <junction x="53.34" y="71.12"/>
 </segment>
@@
 <pinref part="IC1" gate="A" pin="QD"/>
 <wire x1="55.88" y1="68.58" x2="83.82" y2="68.58" width="0.1524" layer="91"/>
-<wire x1="43.18" y1="22.86" x2="55.88" y2="22.86" width="0.1524" layer="91"/>
-<wire x1="55.88" y1="22.86" x2="55.88" y2="68.58" width="0.1524" layer="91"/>
+<wire x1="43.18" y1="20.32" x2="55.88" y2="20.32" width="0.1524" layer="91"/>
+<wire x1="55.88" y1="20.32" x2="55.88" y2="68.58" width="0.1524" layer="91"/>
 <junction x="55.88" y="68.58"/>
 </segment>
@@
 <pinref part="IC1" gate="A" pin="QE"/>
 <wire x1="58.42" y1="66.04" x2="83.82" y2="66.04" width="0.1524" layer="91"/>
-<wire x1="43.18" y1="20.32" x2="58.42" y2="20.32" width="0.1524" layer="91"/>
-<wire x1="58.42" y1="20.32" x2="58.42" y2="66.04" width="0.1524" layer="91"/>
+<wire x1="43.18" y1="17.78" x2="58.42" y2="17.78" width="0.1524" layer="91"/>
+<wire x1="58.42" y1="17.78" x2="58.42" y2="66.04" width="0.1524" layer="91"/>
 <junction x="58.42" y="66.04"/>
 </segment>
@@
 <pinref part="IC1" gate="A" pin="QF"/>
 <wire x1="60.96" y1="63.5" x2="83.82" y2="63.5" width="0.1524" layer="91"/>
-<wire x1="43.18" y1="17.78" x2="60.96" y2="17.78" width="0.1524" layer="91"/>
-<wire x1="60.96" y1="17.78" x2="60.96" y2="63.5" width="0.1524" layer="91"/>
+<wire x1="43.18" y1="15.24" x2="60.96" y2="15.24" width="0.1524" layer="91"/>
+<wire x1="60.96" y1="15.24" x2="60.96" y2="63.5" width="0.1524" layer="91"/>
 <junction x="60.96" y="63.5"/>
 </segment>
@@
 <pinref part="IC1" gate="A" pin="QG"/>
 <wire x1="63.5" y1="60.96" x2="83.82" y2="60.96" width="0.1524" layer="91"/>
-<wire x1="43.18" y1="15.24" x2="63.5" y2="15.24" width="0.1524" layer="91"/>
-<wire x1="63.5" y1="15.24" x2="63.5" y2="60.96" width="0.1524" layer="91"/>
+<wire x1="43.18" y1="12.7" x2="63.5" y2="12.7" width="0.1524" layer="91"/>
+<wire x1="63.5" y1="12.7" x2="63.5" y2="60.96" width="0.1524" layer="91"/>
 <junction x="63.5" y="60.96"/>
 </segment>
@@
 <pinref part="IC1" gate="A" pin="QH"/>
 <wire x1="66.04" y1="58.42" x2="83.82" y2="58.42" width="0.1524" layer="91"/>
-<wire x1="43.18" y1="12.7" x2="66.04" y2="12.7" width="0.1524" layer="91"/>
-<wire x1="66.04" y1="12.7" x2="66.04" y2="58.42" width="0.1524" layer="91"/>
+<wire x1="43.18" y1="10.16" x2="66.04" y2="10.16" width="0.1524" layer="91"/>
+<wire x1="66.04" y1="10.16" x2="66.04" y2="58.42" width="0.1524" layer="91"/>
 <junction x="66.04" y="58.42"/>
 </segment>
@@
 <net name="GND" class="1">
 <segment>
-<pinref part="JP3" gate="G$1" pin="2"/>
+<pinref part="JP5" gate="G$1" pin="2"/>
 <pinref part="GND3" gate="1" pin="GND"/>
 <wire x1="220.98" y1="20.32" x2="203.2" y2="20.32" width="0.1524" layer="91"/>
@@
 <wire x1="203.2" y1="20.32" x2="203.2" y2="43.18" width="0.1524" layer="91"/>
 <junction x="203.2" y="20.32"/>
-<pinref part="JP5" gate="G$1" pin="SLEEVE"/>
+<pinref part="JP4" gate="G$1" pin="SLEEVE"/>
 <wire x1="203.2" y1="43.18" x2="213.36" y2="43.18" width="0.1524" layer="91"/>
 </segment>
@@
 <pinref part="CN1" gate="G$1" pin="GND"/>
 <wire x1="213.36" y1="71.12" x2="213.36" y2="68.58" width="0.1524" layer="91"/>
-<pinref part="GND1" gate="1" pin="GND"/>
+<pinref part="GND2" gate="1" pin="GND"/>
 <wire x1="213.36" y1="68.58" x2="203.2" y2="68.58" width="0.1524" layer="91"/>
 <wire x1="203.2" y1="68.58" x2="203.2" y2="63.5" width="0.1524" layer="91"/>
@@
 </segment>
 <segment>
-<pinref part="GND2" gate="1" pin="GND"/>
+<pinref part="GND1" gate="1" pin="GND"/>
 <pinref part="R1" gate="G$1" pin="1"/>
 <wire x1="119.38" y1="83.82" x2="129.54" y2="83.82" width="0.1524" layer="91"/>
@@
 <net name="N$16" class="0">
 <segment>
-<pinref part="JP4" gate="A" pin="1"/>
 <pinref part="IC1" gate="A" pin="A"/>
-<wire x1="0" y1="30.48" x2="17.78" y2="30.48" width="0.1524" layer="91"/>
+<wire x1="0" y1="27.94" x2="17.78" y2="27.94" width="0.1524" layer="91"/>
+<pinref part="JP3" gate="A" pin="2"/>
 </segment>
 </net>
 <net name="N$29" class="0">
 <segment>
-<pinref part="JP4" gate="A" pin="2"/>
 <pinref part="IC1" gate="A" pin="B"/>
-<wire x1="0" y1="27.94" x2="17.78" y2="27.94" width="0.1524" layer="91"/>
+<wire x1="0" y1="25.4" x2="17.78" y2="25.4" width="0.1524" layer="91"/>
+<pinref part="JP3" gate="A" pin="3"/>
 </segment>
 </net>
 <net name="N$30" class="0">
 <segment>
-<pinref part="JP4" gate="A" pin="4"/>
-<wire x1="0" y1="22.86" x2="12.7" y2="22.86" width="0.1524" layer="91"/>
-<wire x1="12.7" y1="22.86" x2="12.7" y2="12.7" width="0.1524" layer="91"/>
+<wire x1="0" y1="20.32" x2="12.7" y2="20.32" width="0.1524" layer="91"/>
+<wire x1="12.7" y1="20.32" x2="12.7" y2="10.16" width="0.1524" layer="91"/>
 <pinref part="IC1" gate="A" pin="CLR"/>
-<wire x1="12.7" y1="12.7" x2="17.78" y2="12.7" width="0.1524" layer="91"/>
+<wire x1="12.7" y1="10.16" x2="17.78" y2="10.16" width="0.1524" layer="91"/>
+<pinref part="JP3" gate="A" pin="5"/>
 </segment>
 </net>
@@
 <segment>
 <pinref part="IC1" gate="A" pin="CLK"/>
-<wire x1="17.78" y1="17.78" x2="15.24" y2="17.78" width="0.1524" layer="91"/>
-<wire x1="15.24" y1="17.78" x2="15.24" y2="25.4" width="0.1524" layer="91"/>
-<pinref part="JP4" gate="A" pin="3"/>
-<wire x1="15.24" y1="25.4" x2="0" y2="25.4" width="0.1524" layer="91"/>
+<wire x1="17.78" y1="15.24" x2="15.24" y2="15.24" width="0.1524" layer="91"/>
+<wire x1="15.24" y1="15.24" x2="15.24" y2="22.86" width="0.1524" layer="91"/>
+<wire x1="15.24" y1="22.86" x2="0" y2="22.86" width="0.1524" layer="91"/>
+<pinref part="JP3" gate="A" pin="4"/>
 </segment>
 </net>
 <net name="N$32" class="0">
 <segment>
-<pinref part="JP5" gate="G$1" pin="RIGHT"/>
-<pinref part="JP5" gate="G$1" pin="LEFT"/>
+<pinref part="JP4" gate="G$1" pin="RIGHT"/>
+<pinref part="JP4" gate="G$1" pin="LEFT"/>
 <wire x1="213.36" y1="40.64" x2="213.36" y2="38.1" width="0.1524" layer="91"/>
 <pinref part="C1" gate="G$1" pin="-"/>
-<pinref part="JP3" gate="G$1" pin="1"/>
+<pinref part="JP5" gate="G$1" pin="1"/>
 <wire x1="190.5" y1="22.86" x2="195.58" y2="22.86" width="0.1524" layer="91"/>
 <pinref part="R18" gate="G$1" pin="2"/>

Commit message: updates
Parts:
- removed JP4: (no value), SparkFun-Connectors:AUDIO-JACKSPECIAL_POGO_PINS
- added JP6: (no value), KaiBader:AUDIO-JACK-3.5MM
Connections:
- net GND: now also JP6.1; no longer JP4.SLEEVE
- net N$32: now also JP6.2, JP6.3; no longer JP4.LEFT, JP4.RIGHT
Changed lines of the file:
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@@
 <part name="IC1" library="74xx-eu" deviceset="74*164" device="N" technology="HC" value="74HCT164"/>
 <part name="R18" library="rcl" deviceset="R-EU_" device="0204/7" value="47k (optional)"/>
-<part name="JP4" library="SparkFun-Connectors" deviceset="AUDIO-JACK" device="SPECIAL_POGO_PINS"/>
 <part name="JP3" library="pinhead" deviceset="PINHD-1X5" device="" value="SER-IN"/>
+<part name="JP6" library="KaiBader" deviceset="AUDIO-JACK-3.5MM" device=""/>
 </parts>
 <sheets>
@@
 <instance part="IC1" gate="A" x="30.48" y="20.32"/>
 <instance part="R18" gate="G$1" x="195.58" y="17.78" rot="R90"/>
-<instance part="JP4" gate="G$1" x="218.44" y="40.64" rot="MR0"/>
 <instance part="JP3" gate="A" x="-2.54" y="25.4" rot="MR0"/>
+<instance part="JP6" gate="G$1" x="220.98" y="35.56" rot="MR0"/>
 </instances>
 <busses>
@@
 <wire x1="203.2" y1="20.32" x2="203.2" y2="43.18" width="0.1524" layer="91"/>
 <junction x="203.2" y="20.32"/>
-<pinref part="JP4" gate="G$1" pin="SLEEVE"/>
-<wire x1="203.2" y1="43.18" x2="213.36" y2="43.18" width="0.1524" layer="91"/>
+<wire x1="203.2" y1="43.18" x2="210.82" y2="43.18" width="0.1524" layer="91"/>
+<pinref part="JP6" gate="G$1" pin="1"/>
 </segment>
 <segment>
@@
 <net name="N$32" class="0">
 <segment>
-<pinref part="JP4" gate="G$1" pin="RIGHT"/>
-<pinref part="JP4" gate="G$1" pin="LEFT"/>
-<wire x1="213.36" y1="40.64" x2="213.36" y2="38.1" width="0.1524" layer="91"/>
 <pinref part="C1" gate="G$1" pin="-"/>
 <pinref part="JP5" gate="G$1" pin="1"/>
@@
 <junction x="195.58" y="22.86"/>
 <wire x1="205.74" y1="22.86" x2="220.98" y2="22.86" width="0.1524" layer="91"/>
-<wire x1="213.36" y1="38.1" x2="205.74" y2="38.1" width="0.1524" layer="91"/>
-<wire x1="205.74" y1="38.1" x2="205.74" y2="22.86" width="0.1524" layer="91"/>
-<junction x="213.36" y="38.1"/>
+<wire x1="210.82" y1="33.02" x2="205.74" y2="33.02" width="0.1524" layer="91"/>
+<wire x1="205.74" y1="33.02" x2="205.74" y2="22.86" width="0.1524" layer="91"/>
 <junction x="205.74" y="22.86"/>
-</segment>
-</net>
+<pinref part="JP6" gate="G$1" pin="2"/>
+<pinref part="JP6" gate="G$1" pin="3"/>
+<wire x1="210.82" y1="40.64" x2="205.74" y2="40.64" width="0.1524" layer="91"/>
+<wire x1="205.74" y1="40.64" x2="205.74" y2="33.02" width="0.1524" layer="91"/>
+<junction x="205.74" y="33.02"/>
+</segment>
+</net>

Commit message: updates
Connections:
- net VCC: now also JP3.1
Changed lines of the file:
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@@
 <part name="JP3" library="pinhead" deviceset="PINHD-1X5" device="" value="SER-IN"/>
 <part name="JP6" library="KaiBader" deviceset="AUDIO-JACK-3.5MM" device=""/>
+<part name="P+2" library="supply1" deviceset="VCC" device=""/>
 </parts>
 <sheets>
@@
 <instance part="JP3" gate="A" x="-2.54" y="25.4" rot="MR0"/>
 <instance part="JP6" gate="G$1" x="220.98" y="35.56" rot="MR0"/>
+<instance part="P+2" gate="VCC" x="12.7" y="35.56" rot="MR0"/>
 </instances>
 <busses>
@@
 <wire x1="203.2" y1="73.66" x2="203.2" y2="78.74" width="0.1524" layer="91"/>
 </segment>
-</net>
+<segment>
+<pinref part="JP3" gate="A" pin="1"/>
+<pinref part="P+2" gate="VCC" pin="VCC"/>
+<wire x1="0" y1="30.48" x2="12.7" y2="30.48" width="0.1524" layer="91"/>
+<wire x1="12.7" y1="30.48" x2="12.7" y2="33.02" width="0.1524" layer="91"/>
+</segment>
+</net>

Commit message: updates
Parts:
- added JP4: PWR, pinhead:PINHD-1X2
- JP5: device pinhead:PINHD-1X2 -> KaiBader:AUDIO-JACK-3.5MM
- JP6: value (none) -> AUDIO; device KaiBader:AUDIO-JACK-3.5MM -> pinhead:PINHD-1X2
Connections:
- net GND: now also JP4.2, JP5.1, JP6.2; no longer JP5.2, JP6.1
- net N$32: now also JP5.2, JP5.3, JP6.1; no longer JP5.1, JP6.2, JP6.3
- net VCC: now also JP4.1
Changed lines of the file:
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@@
 <part name="JP1" library="pinhead" deviceset="PINHD-1X8" device="" value="PAR-IN"/>
 <part name="JP2" library="pinhead" deviceset="PINHD-1X2" device="" value="LATCH"/>
-<part name="JP5" library="pinhead" deviceset="PINHD-1X2" device=""/>
+<part name="JP6" library="pinhead" deviceset="PINHD-1X2" device="" value="AUDIO"/>
 <part name="CN1" library="KaiBader" deviceset="POWERJACK" device=""/>
-<part name="P+1" library="supply1" deviceset="VCC" device=""/>
+<part name="P+2" library="supply1" deviceset="VCC" device=""/>
 <part name="GND2" library="supply1" deviceset="GND" device=""/>
 <part name="GND1" library="supply1" deviceset="GND" device=""/>
@@
 <part name="R18" library="rcl" deviceset="R-EU_" device="0204/7" value="47k (optional)"/>
 <part name="JP3" library="pinhead" deviceset="PINHD-1X5" device="" value="SER-IN"/>
-<part name="JP6" library="KaiBader" deviceset="AUDIO-JACK-3.5MM" device=""/>
-<part name="P+2" library="supply1" deviceset="VCC" device=""/>
+<part name="JP5" library="KaiBader" deviceset="AUDIO-JACK-3.5MM" device=""/>
+<part name="P+1" library="supply1" deviceset="VCC" device=""/>
+<part name="JP4" library="pinhead" deviceset="PINHD-1X2" device="" value="PWR"/>
 </parts>
 <sheets>
@@
 <instance part="JP1" gate="A" x="-2.54" y="66.04" rot="MR0"/>
 <instance part="JP2" gate="G$1" x="-2.54" y="43.18" rot="MR0"/>
-<instance part="JP5" gate="G$1" x="223.52" y="20.32"/>
+<instance part="JP6" gate="G$1" x="223.52" y="20.32"/>
 <instance part="CN1" gate="G$1" x="215.9" y="66.04" rot="MR0"/>
-<instance part="P+1" gate="VCC" x="203.2" y="81.28" rot="MR0"/>
+<instance part="P+2" gate="VCC" x="203.2" y="81.28" rot="MR0"/>
 <instance part="GND2" gate="1" x="203.2" y="60.96" rot="MR0"/>
 <instance part="GND1" gate="1" x="119.38" y="81.28"/>
@@
 <instance part="R18" gate="G$1" x="195.58" y="17.78" rot="R90"/>
 <instance part="JP3" gate="A" x="-2.54" y="25.4" rot="MR0"/>
-<instance part="JP6" gate="G$1" x="220.98" y="35.56" rot="MR0"/>
-<instance part="P+2" gate="VCC" x="12.7" y="35.56" rot="MR0"/>
+<instance part="JP5" gate="G$1" x="220.98" y="35.56" rot="MR0"/>
+<instance part="P+1" gate="VCC" x="12.7" y="35.56" rot="MR0"/>
+<instance part="JP4" gate="G$1" x="187.96" y="68.58" rot="MR0"/>
 </instances>
 <busses>
@@
 <net name="GND" class="1">
 <segment>
-<pinref part="JP5" gate="G$1" pin="2"/>
+<pinref part="JP6" gate="G$1" pin="2"/>
 <pinref part="GND3" gate="1" pin="GND"/>
 <wire x1="220.98" y1="20.32" x2="203.2" y2="20.32" width="0.1524" layer="91"/>
@@
 <junction x="203.2" y="20.32"/>
 <wire x1="203.2" y1="43.18" x2="210.82" y2="43.18" width="0.1524" layer="91"/>
-<pinref part="JP6" gate="G$1" pin="1"/>
+<pinref part="JP5" gate="G$1" pin="1"/>
 </segment>
 <segment>
@@
 <wire x1="203.2" y1="68.58" x2="203.2" y2="63.5" width="0.1524" layer="91"/>
 <junction x="213.36" y="68.58"/>
+<pinref part="JP4" gate="G$1" pin="2"/>
+<wire x1="190.5" y1="68.58" x2="203.2" y2="68.58" width="0.1524" layer="91"/>
+<junction x="203.2" y="68.58"/>
 </segment>
 <segment>
@@
 <segment>
 <pinref part="CN1" gate="G$1" pin="PWR"/>
-<pinref part="P+1" gate="VCC" pin="VCC"/>
+<pinref part="P+2" gate="VCC" pin="VCC"/>
 <wire x1="213.36" y1="73.66" x2="203.2" y2="73.66" width="0.1524" layer="91"/>
 <wire x1="203.2" y1="73.66" x2="203.2" y2="78.74" width="0.1524" layer="91"/>
+<pinref part="JP4" gate="G$1" pin="1"/>
+<wire x1="190.5" y1="71.12" x2="203.2" y2="71.12" width="0.1524" layer="91"/>
+<wire x1="203.2" y1="71.12" x2="203.2" y2="73.66" width="0.1524" layer="91"/>
+<junction x="203.2" y="73.66"/>
 </segment>
 <segment>
 <pinref part="JP3" gate="A" pin="1"/>
-<pinref part="P+2" gate="VCC" pin="VCC"/>
+<pinref part="P+1" gate="VCC" pin="VCC"/>
 <wire x1="0" y1="30.48" x2="12.7" y2="30.48" width="0.1524" layer="91"/>
 <wire x1="12.7" y1="30.48" x2="12.7" y2="33.02" width="0.1524" layer="91"/>
@@
 <segment>
 <pinref part="C1" gate="G$1" pin="-"/>
-<pinref part="JP5" gate="G$1" pin="1"/>
+<pinref part="JP6" gate="G$1" pin="1"/>
 <wire x1="190.5" y1="22.86" x2="195.58" y2="22.86" width="0.1524" layer="91"/>
 <pinref part="R18" gate="G$1" pin="2"/>
@@
 <wire x1="205.74" y1="33.02" x2="205.74" y2="22.86" width="0.1524" layer="91"/>
 <junction x="205.74" y="22.86"/>
-<pinref part="JP6" gate="G$1" pin="2"/>
-<pinref part="JP6" gate="G$1" pin="3"/>
+<pinref part="JP5" gate="G$1" pin="2"/>
+<pinref part="JP5" gate="G$1" pin="3"/>
 <wire x1="210.82" y1="40.64" x2="205.74" y2="40.64" width="0.1524" layer="91"/>
 <wire x1="205.74" y1="40.64" x2="205.74" y2="33.02" width="0.1524" layer="91"/>
