File: covox.sch (EAGLE design)
At the start: 29 parts, among them CN1 POWERJACK, IC1 74HCT164, IC2 74HCT373

Commit message: updates
Parts:
- JP2: device pinhead:PINHD-1X2 -> pinhead:PINHD-1X3
Connections:
- net GND: now also JP2.1
- net N$26: now also JP2.2; no longer JP2.1
- net N$27: now also JP2.3; no longer JP2.2
Changed lines of the file:
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@@
 <part name="C1" library="rcl" deviceset="CPOL-EU" device="E2-4" value="100nF"/>
 <part name="JP1" library="pinhead" deviceset="PINHD-1X8" device="" value="PAR-IN"/>
-<part name="JP2" library="pinhead" deviceset="PINHD-1X2" device="" value="LATCH"/>
 <part name="JP6" library="pinhead" deviceset="PINHD-1X2" device="" value="AUDIO"/>
 <part name="CN1" library="KaiBader" deviceset="POWERJACK" device=""/>
 <part name="P+2" library="supply1" deviceset="VCC" device=""/>
+<part name="GND3" library="supply1" deviceset="GND" device=""/>
 <part name="GND2" library="supply1" deviceset="GND" device=""/>
-<part name="GND1" library="supply1" deviceset="GND" device=""/>
-<part name="GND3" library="supply1" deviceset="GND" device=""/>
+<part name="GND4" library="supply1" deviceset="GND" device=""/>
 <part name="IC1" library="74xx-eu" deviceset="74*164" device="N" technology="HC" value="74HCT164"/>
 <part name="R18" library="rcl" deviceset="R-EU_" device="0204/7" value="47k (optional)"/>
@@
 <part name="P+1" library="supply1" deviceset="VCC" device=""/>
 <part name="JP4" library="pinhead" deviceset="PINHD-1X2" device="" value="PWR"/>
+<part name="JP2" library="pinhead" deviceset="PINHD-1X3" device="" value="LATCH"/>
+<part name="GND1" library="supply1" deviceset="GND" device=""/>
 </parts>
 <sheets>
@@
 <instance part="C1" gate="G$1" x="185.42" y="22.86" rot="R90"/>
 <instance part="JP1" gate="A" x="-2.54" y="66.04" rot="MR0"/>
-<instance part="JP2" gate="G$1" x="-2.54" y="43.18" rot="MR0"/>
 <instance part="JP6" gate="G$1" x="223.52" y="20.32"/>
 <instance part="CN1" gate="G$1" x="215.9" y="66.04" rot="MR0"/>
 <instance part="P+2" gate="VCC" x="203.2" y="81.28" rot="MR0"/>
-<instance part="GND2" gate="1" x="203.2" y="60.96" rot="MR0"/>
-<instance part="GND1" gate="1" x="119.38" y="81.28"/>
-<instance part="GND3" gate="1" x="203.2" y="5.08"/>
+<instance part="GND3" gate="1" x="203.2" y="60.96" rot="MR0"/>
+<instance part="GND2" gate="1" x="119.38" y="81.28"/>
+<instance part="GND4" gate="1" x="203.2" y="5.08"/>
 <instance part="IC1" gate="A" x="30.48" y="20.32"/>
 <instance part="R18" gate="G$1" x="195.58" y="17.78" rot="R90"/>
@@
 <instance part="P+1" gate="VCC" x="12.7" y="35.56" rot="MR0"/>
 <instance part="JP4" gate="G$1" x="187.96" y="68.58" rot="MR0"/>
+<instance part="JP2" gate="A" x="-2.54" y="43.18" rot="MR0"/>
+<instance part="GND1" gate="1" x="7.62" y="45.72" rot="R90"/>
 </instances>
 <busses>
@@
 <net name="N$26" class="0">
 <segment>
-<pinref part="JP2" gate="G$1" pin="1"/>
-<wire x1="0" y1="45.72" x2="12.7" y2="45.72" width="0.1524" layer="91"/>
-<wire x1="12.7" y1="45.72" x2="12.7" y2="53.34" width="0.1524" layer="91"/>
+<wire x1="0" y1="43.18" x2="12.7" y2="43.18" width="0.1524" layer="91"/>
+<wire x1="12.7" y1="43.18" x2="12.7" y2="53.34" width="0.1524" layer="91"/>
 <pinref part="IC2" gate="A" pin="OC"/>
 <wire x1="12.7" y1="53.34" x2="83.82" y2="53.34" width="0.1524" layer="91"/>
+<pinref part="JP2" gate="A" pin="2"/>
 </segment>
 </net>
 <net name="N$27" class="0">
 <segment>
-<pinref part="JP2" gate="G$1" pin="2"/>
-<wire x1="0" y1="43.18" x2="15.24" y2="43.18" width="0.1524" layer="91"/>
-<wire x1="15.24" y1="43.18" x2="15.24" y2="50.8" width="0.1524" layer="91"/>
+<wire x1="0" y1="40.64" x2="15.24" y2="40.64" width="0.1524" layer="91"/>
+<wire x1="15.24" y1="40.64" x2="15.24" y2="50.8" width="0.1524" layer="91"/>
 <pinref part="IC2" gate="A" pin="ENC"/>
 <wire x1="15.24" y1="50.8" x2="83.82" y2="50.8" width="0.1524" layer="91"/>
+<pinref part="JP2" gate="A" pin="3"/>
 </segment>
 </net>
@@
 <segment>
 <pinref part="JP6" gate="G$1" pin="2"/>
-<pinref part="GND3" gate="1" pin="GND"/>
+<pinref part="GND4" gate="1" pin="GND"/>
 <wire x1="220.98" y1="20.32" x2="203.2" y2="20.32" width="0.1524" layer="91"/>
 <wire x1="203.2" y1="20.32" x2="203.2" y2="12.7" width="0.1524" layer="91"/>
@@
 <pinref part="CN1" gate="G$1" pin="GND"/>
 <wire x1="213.36" y1="71.12" x2="213.36" y2="68.58" width="0.1524" layer="91"/>
-<pinref part="GND2" gate="1" pin="GND"/>
+<pinref part="GND3" gate="1" pin="GND"/>
 <wire x1="213.36" y1="68.58" x2="203.2" y2="68.58" width="0.1524" layer="91"/>
 <wire x1="203.2" y1="68.58" x2="203.2" y2="63.5" width="0.1524" layer="91"/>
@@
 </segment>
 <segment>
-<pinref part="GND1" gate="1" pin="GND"/>
+<pinref part="GND2" gate="1" pin="GND"/>
 <pinref part="R1" gate="G$1" pin="1"/>
 <wire x1="119.38" y1="83.82" x2="129.54" y2="83.82" width="0.1524" layer="91"/>
 </segment>
-</net>
+<segment>
+<pinref part="JP2" gate="A" pin="1"/>
+<pinref part="GND1" gate="1" pin="GND"/>
+<wire x1="0" y1="45.72" x2="5.08" y2="45.72" width="0.1524" layer="91"/>
+</segment>
+</net>

Commit message: updates
Parts:
- JP3: device pinhead:PINHD-1X5 -> pinhead:PINHD-1X4
Connections:
- removed net N$29: IC1A.B, JP3.3
- net N$16: now also IC1A.B, JP3.3; no longer JP3.2
- net N$30: now also JP3.2; no longer JP3.5
Other:
- moved on the sheet: IC1

Commit message: update
Parts:
- CN1: device KaiBader:POWERJACK -> KaiBader:POWERJACK-SLOT
- JP5: value (none) -> AUDIO
Changed lines of the file:
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@@
 <part name="JP1" library="pinhead" deviceset="PINHD-1X8" device="" value="PAR-IN"/>
 <part name="JP6" library="pinhead" deviceset="PINHD-1X2" device="" value="AUDIO"/>
-<part name="CN1" library="KaiBader" deviceset="POWERJACK" device=""/>
 <part name="P+1" library="supply1" deviceset="VCC" device=""/>
 <part name="GND4" library="supply1" deviceset="GND" device=""/>
@@
 <part name="IC1" library="74xx-eu" deviceset="74*164" device="N" technology="HC" value="74HCT164"/>
 <part name="R18" library="rcl" deviceset="R-EU_" device="0204/7" value="47k (optional)"/>
-<part name="JP5" library="KaiBader" deviceset="AUDIO-JACK-3.5MM" device=""/>
+<part name="JP5" library="KaiBader" deviceset="AUDIO-JACK-3.5MM" device="" value="AUDIO"/>
 <part name="JP4" library="pinhead" deviceset="PINHD-1X2" device="" value="PWR"/>
 <part name="JP2" library="pinhead" deviceset="PINHD-1X3" device="" value="LATCH"/>
@@
 <part name="JP3" library="pinhead" deviceset="PINHD-1X4" device="" value="SER-IN"/>
 <part name="P+2" library="supply1" deviceset="VCC" device=""/>
+<part name="CN1" library="KaiBader" deviceset="POWERJACK" device="-SLOT" value="POWERJACK"/>
 </parts>
 <sheets>
@@
 <instance part="JP1" gate="A" x="-2.54" y="66.04" rot="MR0"/>
 <instance part="JP6" gate="G$1" x="223.52" y="20.32"/>
-<instance part="CN1" gate="G$1" x="215.9" y="66.04" rot="MR0"/>
 <instance part="P+1" gate="VCC" x="203.2" y="81.28" rot="MR0"/>
 <instance part="GND4" gate="1" x="203.2" y="60.96" rot="MR0"/>
@@
 <instance part="JP3" gate="A" x="-2.54" y="20.32" rot="MR0"/>
 <instance part="P+2" gate="VCC" x="7.62" y="30.48" rot="MR0"/>
+<instance part="CN1" gate="G$1" x="215.9" y="66.04" rot="MR0"/>
 </instances>
 <busses>
@@
 </segment>
 <segment>
-<pinref part="CN1" gate="G$1" pin="GNDBREAK"/>
-<pinref part="CN1" gate="G$1" pin="GND"/>
 <wire x1="213.36" y1="71.12" x2="213.36" y2="68.58" width="0.1524" layer="91"/>
 <pinref part="GND4" gate="1" pin="GND"/>
 <wire x1="213.36" y1="68.58" x2="203.2" y2="68.58" width="0.1524" layer="91"/>
 <wire x1="203.2" y1="68.58" x2="203.2" y2="63.5" width="0.1524" layer="91"/>
-<junction x="213.36" y="68.58"/>
 <pinref part="JP4" gate="G$1" pin="2"/>
 <wire x1="190.5" y1="68.58" x2="203.2" y2="68.58" width="0.1524" layer="91"/>
 <junction x="203.2" y="68.58"/>
+<pinref part="CN1" gate="G$1" pin="GNDBREAK"/>
+<pinref part="CN1" gate="G$1" pin="GND"/>
+<junction x="213.36" y="68.58"/>
 </segment>
 <segment>
@@
 <net name="VCC" class="1">
 <segment>
-<pinref part="CN1" gate="G$1" pin="PWR"/>
 <pinref part="P+1" gate="VCC" pin="VCC"/>
 <wire x1="213.36" y1="73.66" x2="203.2" y2="73.66" width="0.1524" layer="91"/>
@@
 <wire x1="203.2" y1="71.12" x2="203.2" y2="73.66" width="0.1524" layer="91"/>
 <junction x="203.2" y="73.66"/>
-</segment>
-<segment>
+<pinref part="CN1" gate="G$1" pin="PWR"/>
+</segment>
+<segment>
